File: pcb/tdt4295/VMCU.sch (KiCad schematic (older format))
At the start: 6 parts

Commit message: add indicator LEDs to power supply
Parts:
- gave numbers to parts that had none: 6
Changed lines of the file:
@@
 $EndDescr
 $Comp
-L tdt4295:TS3A4751 U?
+L tdt4295:TS3A4751 U401
 U 1 1 6137905D
 P 5950 3200
-F 0 "U?" H 5600 3750 50  0000 C CNN
+F 0 "U401" H 5600 3750 50  0000 C CNN
 F 1 "TS3A4751" H 6150 3750 50  0000 C CNN
 F 2 "" H 5650 3650 50  0001 C CNN
@@
 $EndComp
 $Comp
-L Device:R R?
+L Device:R R401
 U 1 1 61379BCF
 P 5050 3200
-F 0 "R?" H 5120 3246 50  0000 L CNN
+F 0 "R401" H 5120 3246 50  0000 L CNN
 F 1 "10K" H 5120 3155 50  0000 L CNN
 F 2 "" V 4980 3200 50  0001 C CNN
@@
 $EndComp
 $Comp
-L Device:D D?
+L Device:D D401
 U 1 1 6137F571
 P 7150 2700
-F 0 "D?" H 7150 2917 50  0000 C CNN
+F 0 "D401" H 7150 2917 50  0000 C CNN
 F 1 "D" H 7150 2826 50  0000 C CNN
 F 2 "" H 7150 2700 50  0001 C CNN
@@
 $EndComp
 $Comp
-L Device:D D?
+L Device:D D402
 U 1 1 61380B2E
 P 7150 3350
-F 0 "D?" H 7150 3133 50  0000 C CNN
+F 0 "D402" H 7150 3133 50  0000 C CNN
 F 1 "D" H 7150 3224 50  0000 C CNN
 F 2 "" H 7150 3350 50  0001 C CNN
@@
 	5350 3000 5350 3100
 $Comp
-L power:GND #PWR?
+L power:GND #PWR0403
 U 1 1 61382833
 P 7150 2850
-F 0 "#PWR?" H 7150 2600 50  0001 C CNN
+F 0 "#PWR0403" H 7150 2600 50  0001 C CNN
 F 1 "GND" H 7155 2677 50  0000 C CNN
 F 2 "" H 7150 2850 50  0001 C CNN
@@
 $EndComp
 $Comp
-L power:GND #PWR?
+L power:GND #PWR0404
 U 1 1 6138368D
 P 7150 3500
-F 0 "#PWR?" H 7150 3250 50  0001 C CNN
+F 0 "#PWR0404" H 7150 3250 50  0001 C CNN
 F 1 "GND" H 7155 3327 50  0000 C CNN
 F 2 "" H 7150 3500 50  0001 C CNN
@@
 	5050 3500 5050 3350
 $Comp
-L Device:R R?
+L Device:R R402
 U 1 1 613874B8
 P 5050 4050
-F 0 "R?" H 5120 4096 50  0000 L CNN
+F 0 "R402" H 5120 4096 50  0000 L CNN
 F 1 "180K" H 5120 4005 50  0000 L CNN
 F 2 "" V 4980 4050 50  0001 C CNN
@@
 	5050 3600 5050 3900
 $Comp
-L Device:R R?
+L Device:R R403
 U 1 1 61389242
 P 5350 4050
-F 0 "R?" H 5420 4096 50  0000 L CNN
+F 0 "R403" H 5420 4096 50  0000 L CNN
 F 1 "10M" H 5420 4005 50  0000 L CNN
 F 2 "" V 5280 4050 50  0001 C CNN
@@
 	5350 3400 5350 3800
 $Comp
-L power:GND #PWR?
+L power:GND #PWR0402
 U 1 1 6138E6DA
 P 5350 4300
-F 0 "#PWR?" H 5350 4050 50  0001 C CNN
+F 0 "#PWR0402" H 5350 4050 50  0001 C CNN
 F 1 "GND" H 5355 4127 50  0000 C CNN
 F 2 "" H 5350 4300 50  0001 C CNN
@@
 $EndComp
 $Comp
-L power:GND #PWR?
+L power:GND #PWR0401
 U 1 1 6138F02E
 P 5050 4300
-F 0 "#PWR?" H 5050 4050 50  0001 C CNN
+F 0 "#PWR0401" H 5050 4050 50  0001 C CNN
 F 1 "GND" H 5055 4127 50  0000 C CNN
 F 2 "" H 5050 4300 50  0001 C CNN
