File: pcb/tdt4295/vga.sch (KiCad schematic (older format))
At the start: 33 parts

Commit message: associate symbol components
Parts:
- U401, U402: renamed from U?; footprint PW20 -> SN74ALVC245PWR-footprint:SN74ALVC245PWR
- gave numbers to parts that had none: 31
