File: pcb/tdt4295/tdt4295.sch (KiCad schematic (older format))
At the start: 44 parts, among them J101 ARM 20 Pin Debug Header, J102 SD_Card, J103 MCU USART1 Header, J104 MCU GPIO Header, U101 EFM32GG12B810F1024GQ64, U102 COM-09032 Joystick, U103 COM-09032 Joystick, Y101 48MHz

Commit message: pcb: Added some more footprints/part numbers
Parts:
- C103, C107, C110, C111, C112: footprint (none) -> Capacitor_SMD:C_0603_1608Metric_Pad1.08x0.95mm_HandSolder; Component name (none) -> CL10B104KA8NNNC; DK_Datasheet_Link (none) -> https://www.digikey.no/product-detail/en/samsung-electro-me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
- C105, C106, C113: footprint (none) -> Capacitor_SMD:C_0603_1608Metric_Pad1.08x0.95mm_HandSolder; Component name (none) -> CL10A106KQ8NNNC; DK_Datasheet_Link (none) -> https://www.digikey.no/product-detail/en/samsung-electro-me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
- C108, C109: footprint (none) -> Capacitor_SMD:C_0603_1608Metric_Pad1.08x0.95mm_HandSolder; Component name (none) -> CL21B105KOFNNNE; DK_Datasheet_Link (none) -> https://www.digikey.no/product-detail/en/samsung-electro-me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
- Y101: footprint (none) -> Crystal:Crystal_SMD_2016-4Pin_2.0x1.6mm
Changed lines of the file:
@@
 F 0 "Y101" H 4350 4500 50  0000 L CNN
 F 1 "48MHz" H 4350 4250 50  0000 L CNN
-F 2 "" H 4250 4350 50  0001 C CNN
+F 2 "Crystal:Crystal_SMD_2016-4Pin_2.0x1.6mm" H 4250 4350 50  0001 C CNN
 F 3 "https://www.farnell.com/datasheets/1883673.pdf" H 4250 4350 50  0001 C CNN
 	1    4250 4350
@@
 F 0 "C110" H 9715 2296 50  0000 L CNN
 F 1 "0.1uF" H 9715 2205 50  0000 L CNN
-F 2 "" H 9638 2100 50  0001 C CNN
+F 2 "Capacitor_SMD:C_0603_1608Metric_Pad1.08x0.95mm_HandSolder" H 9638 2100 50  0001 C CNN
 F 3 "~" H 9600 2250 50  0001 C CNN
+F 4 "CL10B104KA8NNNC" H 9600 2250 50  0001 C CNN "Component name"
+F 5 "https://www.digikey.no/product-detail/en/samsung-electro-mechanics/CL10B104KA8NNNC/1276-1006-1-ND/3889092" H 9600 2250 50  0001 C CNN "DK_Datasheet_Link"
 	1    9600 2250
 	1    0    0    -1
@@
 F 0 "C103" H 5200 4550 50  0000 L CNN
 F 1 "0.1uF" H 5200 4350 50  0000 L CNN
-F 2 "" H 5238 4300 50  0001 C CNN
+F 2 "Capacitor_SMD:C_0603_1608Metric_Pad1.08x0.95mm_HandSolder" H 5238 4300 50  0001 C CNN
 F 3 "~" H 5200 4450 50  0001 C CNN
+F 4 "CL10B104KA8NNNC" H 5200 4450 50  0001 C CNN "Component name"
+F 5 "https://www.digikey.no/product-detail/en/samsung-electro-mechanics/CL10B104KA8NNNC/1276-1006-1-ND/3889092" H 5200 4450 50  0001 C CNN "DK_Datasheet_Link"
 	1    5200 4450
 	1    0    0    -1
@@
 F 0 "C107" H 5900 2550 50  0000 L CNN
 F 1 "0.1uF" H 5900 2350 50  0000 L CNN
-F 2 "" H 5888 2300 50  0001 C CNN
+F 2 "Capacitor_SMD:C_0603_1608Metric_Pad1.08x0.95mm_HandSolder" H 5888 2300 50  0001 C CNN
 F 3 "~" H 5850 2450 50  0001 C CNN
+F 4 "CL10B104KA8NNNC" H 5850 2450 50  0001 C CNN "Component name"
+F 5 "https://www.digikey.no/product-detail/en/samsung-electro-mechanics/CL10B104KA8NNNC/1276-1006-1-ND/3889092" H 5850 2450 50  0001 C CNN "DK_Datasheet_Link"
 	1    5850 2450
 	1    0    0    -1
@@
 F 0 "C105" H 5600 2550 50  0000 L CNN
 F 1 "10uF" H 5600 2350 50  0000 L CNN
-F 2 "" H 5588 2300 50  0001 C CNN
+F 2 "Capacitor_SMD:C_0603_1608Metric_Pad1.08x0.95mm_HandSolder" H 5588 2300 50  0001 C CNN
 F 3 "~" H 5550 2450 50  0001 C CNN
+F 4 "CL10A106KQ8NNNC" H 5550 2450 50  0001 C CNN "Component name"
+F 5 "https://www.digikey.no/product-detail/en/samsung-electro-mechanics/CL10A106KQ8NNNC/1276-1038-1-ND/3889124" H 5550 2450 50  0001 C CNN "DK_Datasheet_Link"
 	1    5550 2450
 	1    0    0    -1
@@
 F 0 "C109" H 9550 4300 50  0000 L CNN
 F 1 "1uF" H 9550 4100 50  0000 L CNN
-F 2 "" H 9588 4050 50  0001 C CNN
-F 3 "~" H 9550 4200 50  0001 C CNN
+F 2 "Capacitor_SMD:C_0603_1608Metric_Pad1.08x0.95mm_HandSolder" H 9588 4050 50  0001 C CNN
+F 3 "www.samsungsem.com/kr/support/product-search/mlcc/CL21B105KOFNNNE.jsp" H 9550 4200 50  0001 C CNN
+F 4 "CL21B105KOFNNNE" H 9550 4200 50  0001 C CNN "Component name"
+F 5 "https://www.digikey.no/product-detail/en/samsung-electro-mechanics/CL21B105KOFNNNE/1276-1026-1-ND/3889112" H 9550 4200 50  0001 C CNN "DK_Datasheet_Link"
 	1    9550 4200
 	1    0    0    -1
@@
 F 0 "C106" H 5750 4550 50  0000 L CNN
 F 1 "10uF" H 5750 4350 50  0000 L CNN
-F 2 "" H 5788 4300 50  0001 C CNN
+F 2 "Capacitor_SMD:C_0603_1608Metric_Pad1.08x0.95mm_HandSolder" H 5788 4300 50  0001 C CNN
 F 3 "~" H 5750 4450 50  0001 C CNN
+F 4 "CL10A106KQ8NNNC" H 5750 4450 50  0001 C CNN "Component name"
+F 5 "https://www.digikey.no/product-detail/en/samsung-electro-mechanics/CL10A106KQ8NNNC/1276-1038-1-ND/3889124" H 5750 4450 50  0001 C CNN "DK_Datasheet_Link"
 	1    5750 4450
 	1    0    0    -1
@@
 F 0 "C113" H 10400 4300 50  0000 L CNN
 F 1 "10uF" H 10400 4100 50  0000 L CNN
-F 2 "" H 10438 4050 50  0001 C CNN
+F 2 "Capacitor_SMD:C_0603_1608Metric_Pad1.08x0.95mm_HandSolder" H 10438 4050 50  0001 C CNN
 F 3 "~" H 10400 4200 50  0001 C CNN
+F 4 "CL10A106KQ8NNNC" H 10400 4200 50  0001 C CNN "Component name"
+F 5 "https://www.digikey.no/product-detail/en/samsung-electro-mechanics/CL10A106KQ8NNNC/1276-1038-1-ND/3889124" H 10400 4200 50  0001 C CNN "DK_Datasheet_Link"
 	1    10400 4200
 	1    0    0    -1
@@
 F 0 "C112" H 10150 4300 50  0000 L CNN
 F 1 "0.1uF" H 10150 4100 50  0000 L CNN
-F 2 "" H 10188 4050 50  0001 C CNN
+F 2 "Capacitor_SMD:C_0603_1608Metric_Pad1.08x0.95mm_HandSolder" H 10188 4050 50  0001 C CNN
 F 3 "~" H 10150 4200 50  0001 C CNN
+F 4 "CL10B104KA8NNNC" H 10150 4200 50  0001 C CNN "Component name"
+F 5 "https://www.digikey.no/product-detail/en/samsung-electro-mechanics/CL10B104KA8NNNC/1276-1006-1-ND/3889092" H 10150 4200 50  0001 C CNN "DK_Datasheet_Link"
 	1    10150 4200
 	1    0    0    -1
@@
 F 0 "C111" H 9850 4300 50  0000 L CNN
 F 1 "0.1uF" H 9850 4100 50  0000 L CNN
-F 2 "" H 9888 4050 50  0001 C CNN
+F 2 "Capacitor_SMD:C_0603_1608Metric_Pad1.08x0.95mm_HandSolder" H 9888 4050 50  0001 C CNN
 F 3 "~" H 9850 4200 50  0001 C CNN
+F 4 "CL10B104KA8NNNC" H 9850 4200 50  0001 C CNN "Component name"
+F 5 "https://www.digikey.no/product-detail/en/samsung-electro-mechanics/CL10B104KA8NNNC/1276-1006-1-ND/3889092" H 9850 4200 50  0001 C CNN "DK_Datasheet_Link"
 	1    9850 4200
 	1    0    0    -1
@@
 F 0 "C108" H 9600 3650 50  0000 L CNN
 F 1 "1uF" H 9600 3550 50  0000 L CNN
-F 2 "" H 9538 3450 50  0001 C CNN
-F 3 "~" H 9500 3600 50  0001 C CNN
+F 2 "Capacitor_SMD:C_0603_1608Metric_Pad1.08x0.95mm_HandSolder" H 9538 3450 50  0001 C CNN
+F 3 "www.samsungsem.com/kr/support/product-search/mlcc/CL21B105KOFNNNE.jsp" H 9500 3600 50  0001 C CNN
+F 4 "CL21B105KOFNNNE" H 9500 3600 50  0001 C CNN "Component name"
+F 5 "https://www.digikey.no/product-detail/en/samsung-electro-mechanics/CL21B105KOFNNNE/1276-1026-1-ND/3889112" H 9500 3600 50  0001 C CNN "DK_Datasheet_Link"
 	1    9500 3600
 	1    0    0    -1

Commit message: pcb: footprints/components for everything but inductors
Parts:
- C101, C102: Category C1210C107M9PACTU -> (none); Component name (none) -> C1210C107M9PACTU
- C103, C105, C106, C107, C108, C109, C110, C111, C112, C113: DK_Detail_Page (none) -> https://www.digikey.no/product-detail/en/samsung-electro-me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
- C104: footprint (none) -> Capacitor_SMD:C_0603_1608Metric_Pad1.08x0.95mm_HandSolder; Component name (none) -> CL10B103KB8NNNC; DK_Datasheet_Link (none) -> https://media.digikey.com/pdf/Data%20Sheets/Samsung%20PDFs/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; DK_Detail_Page (none) -> https://www.digikey.no/product-detail/en/samsung-electro-me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
- D101, D102, D103, D104: footprint (none) -> Diode_SMD:D_0805_2012Metric_Pad1.15x1.40mm_HandSolder
- J102: footprint (none) -> Connector_Card:microSD_HC_Wuerth_693072010801
Changed lines of the file:
@@
 F 2 "Capacitor_SMD:C_1210_3225Metric_Pad1.33x2.70mm_HandSolder" H 4738 4350 50  0001 C CNN
 F 3 "https://api.kemet.com/component-edge/download/specsheet/C1210C107M9PACTU.pdf" H 4700 4500 50  0001 C CNN
-F 4 "C1210C107M9PACTU" H 4700 4500 50  0001 C CNN "Category"
+F 4 "" H 4700 4500 50  0001 C CNN "Category"
 F 5 "https://no.farnell.com/kemet/c1210c107m9pactu/cap-100-f-6-3v-20-x5r-1210/dp/1108328?st=c1210c107m9pactu" H 4700 4500 50  0001 C CNN "DK_Detail_Page"
+F 6 "C1210C107M9PACTU" H 4700 4500 50  0001 C CNN "Component name"
 	1    4700 4500
 	1    0    0    -1
@@
 F 2 "Capacitor_SMD:C_1210_3225Metric_Pad1.33x2.70mm_HandSolder" H 3838 4350 50  0001 C CNN
 F 3 "https://api.kemet.com/component-edge/download/specsheet/C1210C107M9PACTU.pdf" H 3800 4500 50  0001 C CNN
-F 4 "C1210C107M9PACTU" H 3800 4500 50  0001 C CNN "Category"
+F 4 "" H 3800 4500 50  0001 C CNN "Category"
 F 5 "https://no.farnell.com/kemet/c1210c107m9pactu/cap-100-f-6-3v-20-x5r-1210/dp/1108328?st=c1210c107m9pactu" H 3800 4500 50  0001 C CNN "DK_Detail_Page"
+F 6 "C1210C107M9PACTU" H 3800 4500 50  0001 C CNN "Component name"
 	1    3800 4500
 	1    0    0    -1
@@
 F 0 "J102" H 12500 5465 50  0000 C CNN
 F 1 "SD_Card" H 12500 5374 50  0000 C CNN
-F 2 "" H 12500 4800 50  0001 C CNN
+F 2 "Connector_Card:microSD_HC_Wuerth_693072010801" H 12500 4800 50  0001 C CNN
 F 3 "http://portal.fciconnect.com/Comergent//fci/drawing/10067847.pdf" H 12500 4800 50  0001 C CNN
 	1    12500 4800
@@
 F 4 "CL10B104KA8NNNC" H 9600 2250 50  0001 C CNN "Component name"
 F 5 "https://www.digikey.no/product-detail/en/samsung-electro-mechanics/CL10B104KA8NNNC/1276-1006-1-ND/3889092" H 9600 2250 50  0001 C CNN "DK_Datasheet_Link"
+F 6 "https://www.digikey.no/product-detail/en/samsung-electro-mechanics/CL10B104KA8NNNC/1276-1006-1-ND/3889092" H 9600 2250 50  0001 C CNN "DK_Detail_Page"
 	1    9600 2250
 	1    0    0    -1
@@
 F 4 "CL10B104KA8NNNC" H 5200 4450 50  0001 C CNN "Component name"
 F 5 "https://www.digikey.no/product-detail/en/samsung-electro-mechanics/CL10B104KA8NNNC/1276-1006-1-ND/3889092" H 5200 4450 50  0001 C CNN "DK_Datasheet_Link"
+F 6 "https://www.digikey.no/product-detail/en/samsung-electro-mechanics/CL10B104KA8NNNC/1276-1006-1-ND/3889092" H 5200 4450 50  0001 C CNN "DK_Detail_Page"
 	1    5200 4450
 	1    0    0    -1
@@
 F 4 "CL10B104KA8NNNC" H 5850 2450 50  0001 C CNN "Component name"
 F 5 "https://www.digikey.no/product-detail/en/samsung-electro-mechanics/CL10B104KA8NNNC/1276-1006-1-ND/3889092" H 5850 2450 50  0001 C CNN "DK_Datasheet_Link"
+F 6 "https://www.digikey.no/product-detail/en/samsung-electro-mechanics/CL10B104KA8NNNC/1276-1006-1-ND/3889092" H 5850 2450 50  0001 C CNN "DK_Detail_Page"
 	1    5850 2450
 	1    0    0    -1
@@
 F 4 "CL10A106KQ8NNNC" H 5550 2450 50  0001 C CNN "Component name"
 F 5 "https://www.digikey.no/product-detail/en/samsung-electro-mechanics/CL10A106KQ8NNNC/1276-1038-1-ND/3889124" H 5550 2450 50  0001 C CNN "DK_Datasheet_Link"
+F 6 "https://www.digikey.no/product-detail/en/samsung-electro-mechanics/CL10A106KQ8NNNC/1276-1038-1-ND/3889124" H 5550 2450 50  0001 C CNN "DK_Detail_Page"
 	1    5550 2450
 	1    0    0    -1
@@
 F 4 "CL21B105KOFNNNE" H 9550 4200 50  0001 C CNN "Component name"
 F 5 "https://www.digikey.no/product-detail/en/samsung-electro-mechanics/CL21B105KOFNNNE/1276-1026-1-ND/3889112" H 9550 4200 50  0001 C CNN "DK_Datasheet_Link"
+F 6 "https://www.digikey.no/product-detail/en/samsung-electro-mechanics/CL21B105KOFNNNE/1276-1026-1-ND/3889112" H 9550 4200 50  0001 C CNN "DK_Detail_Page"
 	1    9550 4200
 	1    0    0    -1
@@
 F 0 "C104" H 5500 4550 50  0000 L CNN
 F 1 "10nF" H 5500 4350 50  0000 L CNN
-F 2 "" H 5538 4300 50  0001 C CNN
+F 2 "Capacitor_SMD:C_0603_1608Metric_Pad1.08x0.95mm_HandSolder" H 5538 4300 50  0001 C CNN
 F 3 "~" H 5500 4450 50  0001 C CNN
+F 4 "CL10B103KB8NNNC" H 5500 4450 50  0001 C CNN "Component name"
+F 5 "https://media.digikey.com/pdf/Data%20Sheets/Samsung%20PDFs/CL10B103KB8NNNC_Spec.pdf" H 5500 4450 50  0001 C CNN "DK_Datasheet_Link"
+F 6 "https://www.digikey.no/product-detail/en/samsung-electro-mechanics/CL10B103KB8NNNC/1276-1009-1-ND/3889095" H 5500 4450 50  0001 C CNN "DK_Detail_Page"
 	1    5500 4450
 	1    0    0    -1
@@
 F 4 "CL10A106KQ8NNNC" H 5750 4450 50  0001 C CNN "Component name"
 F 5 "https://www.digikey.no/product-detail/en/samsung-electro-mechanics/CL10A106KQ8NNNC/1276-1038-1-ND/3889124" H 5750 4450 50  0001 C CNN "DK_Datasheet_Link"
+F 6 "https://www.digikey.no/product-detail/en/samsung-electro-mechanics/CL10A106KQ8NNNC/1276-1038-1-ND/3889124" H 5750 4450 50  0001 C CNN "DK_Detail_Page"
 	1    5750 4450
 	1    0    0    -1
@@
 F 4 "CL10A106KQ8NNNC" H 10400 4200 50  0001 C CNN "Component name"
 F 5 "https://www.digikey.no/product-detail/en/samsung-electro-mechanics/CL10A106KQ8NNNC/1276-1038-1-ND/3889124" H 10400 4200 50  0001 C CNN "DK_Datasheet_Link"
+F 6 "https://www.digikey.no/product-detail/en/samsung-electro-mechanics/CL10A106KQ8NNNC/1276-1038-1-ND/3889124" H 10400 4200 50  0001 C CNN "DK_Detail_Page"
 	1    10400 4200
 	1    0    0    -1
@@
 F 4 "CL10B104KA8NNNC" H 10150 4200 50  0001 C CNN "Component name"
 F 5 "https://www.digikey.no/product-detail/en/samsung-electro-mechanics/CL10B104KA8NNNC/1276-1006-1-ND/3889092" H 10150 4200 50  0001 C CNN "DK_Datasheet_Link"
+F 6 "https://www.digikey.no/product-detail/en/samsung-electro-mechanics/CL10B104KA8NNNC/1276-1006-1-ND/3889092" H 10150 4200 50  0001 C CNN "DK_Detail_Page"
 	1    10150 4200
 	1    0    0    -1
@@
 F 4 "CL10B104KA8NNNC" H 9850 4200 50  0001 C CNN "Component name"
 F 5 "https://www.digikey.no/product-detail/en/samsung-electro-mechanics/CL10B104KA8NNNC/1276-1006-1-ND/3889092" H 9850 4200 50  0001 C CNN "DK_Datasheet_Link"
+F 6 "https://www.digikey.no/product-detail/en/samsung-electro-mechanics/CL10B104KA8NNNC/1276-1006-1-ND/3889092" H 9850 4200 50  0001 C CNN "DK_Detail_Page"
 	1    9850 4200
 	1    0    0    -1
@@
 F 4 "CL21B105KOFNNNE" H 9500 3600 50  0001 C CNN "Component name"
 F 5 "https://www.digikey.no/product-detail/en/samsung-electro-mechanics/CL21B105KOFNNNE/1276-1026-1-ND/3889112" H 9500 3600 50  0001 C CNN "DK_Datasheet_Link"
+F 6 "https://www.digikey.no/product-detail/en/samsung-electro-mechanics/CL21B105KOFNNNE/1276-1026-1-ND/3889112" H 9500 3600 50  0001 C CNN "DK_Detail_Page"
 	1    9500 3600
 	1    0    0    -1
@@
 F 0 "D101" V 3839 1832 50  0000 R CNN
 F 1 "LED" V 3748 1832 50  0000 R CNN
-F 2 "" H 3800 1950 50  0001 C CNN
+F 2 "Diode_SMD:D_0805_2012Metric_Pad1.15x1.40mm_HandSolder" H 3800 1950 50  0001 C CNN
 F 3 "~" H 3800 1950 50  0001 C CNN
 	1    3800 1950
@@
 F 0 "D102" V 4189 1832 50  0000 R CNN
 F 1 "LED" V 4098 1832 50  0000 R CNN
-F 2 "" H 4150 1950 50  0001 C CNN
+F 2 "Diode_SMD:D_0805_2012Metric_Pad1.15x1.40mm_HandSolder" H 4150 1950 50  0001 C CNN
 F 3 "~" H 4150 1950 50  0001 C CNN
 	1    4150 1950
@@
 F 0 "D103" V 4539 1832 50  0000 R CNN
 F 1 "LED" V 4448 1832 50  0000 R CNN
-F 2 "" H 4500 1950 50  0001 C CNN
+F 2 "Diode_SMD:D_0805_2012Metric_Pad1.15x1.40mm_HandSolder" H 4500 1950 50  0001 C CNN
 F 3 "~" H 4500 1950 50  0001 C CNN
 	1    4500 1950
@@
 F 0 "D104" V 4889 1832 50  0000 R CNN
 F 1 "LED" V 4798 1832 50  0000 R CNN
-F 2 "" H 4850 1950 50  0001 C CNN
+F 2 "Diode_SMD:D_0805_2012Metric_Pad1.15x1.40mm_HandSolder" H 4850 1950 50  0001 C CNN
 F 3 "~" H 4850 1950 50  0001 C CNN
 	1    4850 1950
