File: pcb/tdt4295/tdt4295.sch (KiCad schematic (older format))
At the start: 40 parts, among them J101 ARM 20 Pin Debug Header, J102 MCU USART1 Header, J103 DM1AA-SF-PEJ(21), J104 MCU GPIO Header, U101 EFM32GG12B810F1024GQ64, U102 COM-09032 Joystick, U103 COM-09032 Joystick, Y101 48MHz

Commit message: associate component links with (almost) every component
Parts:
- D101, D102, D103, D104: footprint LED_SMD:LED_2816_7142Metric_Pad3.20x4.45mm_HandSolder -> LED_SMD:LED_1206_3216Metric_Pad1.42x1.75mm_HandSolder; Component name (none) -> 150120BS75000; DK_Detail_Page (none) -> https://www.digikey.no/product-detail/no/w%C3%BCrth-elektro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
- J101: footprint Connector_PinHeader_2.54mm:PinHeader_2x10_P2.54mm_Vertical -> Connector_PinHeader_1.27mm:PinHeader_2x10_P1.27mm_Vertical_SMD; Component name (none) -> FTSH-110-01-L-DV-K-TR; DK_Detail_Page (none) -> https://www.digikey.no/product-detail/en/samtec-inc/FTSH-11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
- J102: footprint Connector_PinHeader_2.54mm:PinHeader_2x06_P2.54mm_Vertical -> Connector_PinHeader_2.54mm:PinHeader_2x06_P2.54mm_Vertical_SMD; Component name (none) -> 0015910120; DK_Detail_Page (none) -> https://www.digikey.no/product-detail/en/molex/0015910120/W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
- J103: footprint HRS_DM1AA-SF-PEJ(21) -> DM1AA-SF-PEJ_21:HRS_DM1AA-SF-PEJ(21); Component name (none) -> DM1AA-SF-PEJ-21; DK_Detail_Page (none) -> https://www.digikey.no/product-detail/no/hirose-electric-co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
- J104: footprint Connector_PinSocket_2.54mm:PinSocket_1x07_P2.54mm_Vertical -> Connector_PinSocket_2.54mm:PinSocket_1x07_P2.54mm_Vertical_SMD_Pin1Right; Component name (none) -> 0878980726; DK_Detail_Page (none) -> https://www.digikey.no/product-detail/en/molex/0878980726/W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
- R105, R106: DK_Detail_Page (none) -> https://www.digikey.no/product-detail/no/te-connectivity-pa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
- U102, U103: Component name (none) -> COM-09032; DK_Detail_Page (none) -> https://www.digikey.no/product-detail/no/sparkfun-electroni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
- Y101: Component name (none) -> ABM11-48.000MHZ-D2X-T3; DK_Detail_Page (none) -> https://no.farnell.com/abracon/abm11-48-000mhz-d2x-t3/cryst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
Changed lines of the file:
@@
 F 2 "Crystal:Crystal_SMD_2016-4Pin_2.0x1.6mm" H 4250 4350 50  0001 C CNN
 F 3 "https://www.farnell.com/datasheets/1883673.pdf" H 4250 4350 50  0001 C CNN
+F 4 "ABM11-48.000MHZ-D2X-T3" H 4250 4350 50  0001 C CNN "Component name"
+F 5 "https://no.farnell.com/abracon/abm11-48-000mhz-d2x-t3/crystal-48mhz-10pf-2-x-1-6mm/dp/2467782RL?st=krystall" H 4250 4350 50  0001 C CNN "DK_Detail_Page"
 	1    4250 4350
 	1    0    0    -1
@@
 F 0 "J101" V 11100 1950 50  0000 L CNN
 F 1 "ARM 20 Pin Debug Header" V 11000 1950 50  0000 L CNN
-F 2 "Connector_PinHeader_2.54mm:PinHeader_2x10_P2.54mm_Vertical" H 10900 1450 50  0001 C CNN
+F 2 "Connector_PinHeader_1.27mm:PinHeader_2x10_P1.27mm_Vertical_SMD" H 10900 1450 50  0001 C CNN
 F 3 "~" H 10900 1450 50  0001 C CNN
+F 4 "FTSH-110-01-L-DV-K-TR" H 10900 1450 50  0001 C CNN "Component name"
+F 5 "https://www.digikey.no/product-detail/en/samtec-inc/FTSH-110-01-L-DV-K-TR/SAM13960TR-ND/6693931" H 10900 1450 50  0001 C CNN "DK_Detail_Page"
 	1    10900 1450
 	0    1    -1   0
@@
 F 3 "https://www.te.com/commerce/DocumentDelivery/DDEController?Action=srchrtrv&DocNm=9-1773463-7&DocType=DS&DocLang=English" H 9100 3200 50  0001 C CNN
 F 4 "352215RFT" H 9100 3200 50  0001 C CNN "Category"
+F 5 "https://www.digikey.no/product-detail/no/te-connectivity-passive-product/352215RFT/A121147CT-ND/5245204" H 9100 3200 50  0001 C CNN "DK_Detail_Page"
 	1    9100 3200
 	0    1    1    0
@@
 F 3 "https://www.te.com/commerce/DocumentDelivery/DDEController?Action=srchrtrv&DocNm=9-1773463-7&DocType=DS&DocLang=English" H 9100 3300 50  0001 C CNN
 F 4 "352215RFT" H 9100 3300 50  0001 C CNN "Category"
+F 5 "https://www.digikey.no/product-detail/no/te-connectivity-passive-product/352215RFT/A121147CT-ND/5245204" H 9100 3300 50  0001 C CNN "DK_Detail_Page"
 	1    9100 3300
 	0    1    1    0
@@
 F 0 "D101" V 3839 1832 50  0000 R CNN
 F 1 "LED" V 3748 1832 50  0000 R CNN
-F 2 "LED_SMD:LED_2816_7142Metric_Pad3.20x4.45mm_HandSolder" H 3800 1950 50  0001 C CNN
+F 2 "LED_SMD:LED_1206_3216Metric_Pad1.42x1.75mm_HandSolder" H 3800 1950 50  0001 C CNN
 F 3 "~" H 3800 1950 50  0001 C CNN
+F 4 "150120BS75000" H 3800 1950 50  0001 C CNN "Component name"
+F 5 "https://www.digikey.no/product-detail/no/w%C3%BCrth-elektronik/150120BS75000/732-4989-1-ND/4489931" H 3800 1950 50  0001 C CNN "DK_Detail_Page"
 	1    3800 1950
 	0    -1   -1   0
@@
 F 0 "D102" V 4189 1832 50  0000 R CNN
 F 1 "LED" V 4098 1832 50  0000 R CNN
-F 2 "LED_SMD:LED_2816_7142Metric_Pad3.20x4.45mm_HandSolder" H 4150 1950 50  0001 C CNN
+F 2 "LED_SMD:LED_1206_3216Metric_Pad1.42x1.75mm_HandSolder" H 4150 1950 50  0001 C CNN
 F 3 "~" H 4150 1950 50  0001 C CNN
+F 4 "150120BS75000" H 4150 1950 50  0001 C CNN "Component name"
+F 5 "https://www.digikey.no/product-detail/no/w%C3%BCrth-elektronik/150120BS75000/732-4989-1-ND/4489931" H 4150 1950 50  0001 C CNN "DK_Detail_Page"
 	1    4150 1950
 	0    -1   -1   0
@@
 F 0 "D103" V 4539 1832 50  0000 R CNN
 F 1 "LED" V 4448 1832 50  0000 R CNN
-F 2 "LED_SMD:LED_2816_7142Metric_Pad3.20x4.45mm_HandSolder" H 4500 1950 50  0001 C CNN
+F 2 "LED_SMD:LED_1206_3216Metric_Pad1.42x1.75mm_HandSolder" H 4500 1950 50  0001 C CNN
 F 3 "~" H 4500 1950 50  0001 C CNN
+F 4 "150120BS75000" H 4500 1950 50  0001 C CNN "Component name"
+F 5 "https://www.digikey.no/product-detail/no/w%C3%BCrth-elektronik/150120BS75000/732-4989-1-ND/4489931" H 4500 1950 50  0001 C CNN "DK_Detail_Page"
 	1    4500 1950
 	0    -1   -1   0
@@
 F 0 "D104" V 4889 1832 50  0000 R CNN
 F 1 "LED" V 4798 1832 50  0000 R CNN
-F 2 "LED_SMD:LED_2816_7142Metric_Pad3.20x4.45mm_HandSolder" H 4850 1950 50  0001 C CNN
+F 2 "LED_SMD:LED_1206_3216Metric_Pad1.42x1.75mm_HandSolder" H 4850 1950 50  0001 C CNN
 F 3 "~" H 4850 1950 50  0001 C CNN
+F 4 "150120BS75000" H 4850 1950 50  0001 C CNN "Component name"
+F 5 "https://www.digikey.no/product-detail/no/w%C3%BCrth-elektronik/150120BS75000/732-4989-1-ND/4489931" H 4850 1950 50  0001 C CNN "DK_Detail_Page"
 	1    4850 1950
 	0    -1   -1   0
@@
 F 6 "Manufacturer Recommendations" H 15150 3100 50  0001 L BNN "STANDARD"
 F 7 "N/A" H 15150 2900 50  0001 L BNN "PARTREV"
+F 8 "COM-09032" H 14850 3300 50  0001 C CNN "Component name"
+F 9 "https://www.digikey.no/product-detail/no/sparkfun-electronics/COM-09032/1568-1526-ND/6823623" H 14850 3300 50  0001 C CNN "DK_Detail_Page"
 	1    14850 3300
 	1    0    0    -1
@@
 F 6 "Manufacturer Recommendations" H 15150 4500 50  0001 L BNN "STANDARD"
 F 7 "N/A" H 15150 4300 50  0001 L BNN "PARTREV"
+F 8 "COM-09032" H 14850 4700 50  0001 C CNN "Component name"
+F 9 "https://www.digikey.no/product-detail/no/sparkfun-electronics/COM-09032/1568-1526-ND/6823623" H 14850 4700 50  0001 C CNN "DK_Detail_Page"
 	1    14850 4700
 	1    0    0    -1
@@
 F 0 "J104" H 12630 3442 50  0000 L CNN
 F 1 "MCU GPIO Header" H 12630 3351 50  0000 L CNN
-F 2 "Connector_PinSocket_2.54mm:PinSocket_1x07_P2.54mm_Vertical" H 12550 3400 50  0001 C CNN
+F 2 "Connector_PinSocket_2.54mm:PinSocket_1x07_P2.54mm_Vertical_SMD_Pin1Right" H 12550 3400 50  0001 C CNN
 F 3 "~" H 12550 3400 50  0001 C CNN
+F 4 "0878980726" H 12550 3400 50  0001 C CNN "Component name"
+F 5 "https://www.digikey.no/product-detail/en/molex/0878980726/WM20569-ND/3264913" H 12550 3400 50  0001 C CNN "DK_Detail_Page"
 	1    12550 3400
 	1    0    0    -1
@@
 F 0 "J103" H 12200 5517 50  0000 C CNN
 F 1 "DM1AA-SF-PEJ(21)" H 12200 5426 50  0000 C CNN
-F 2 "HRS_DM1AA-SF-PEJ(21)" H 12200 4850 50  0001 L BNN
+F 2 "DM1AA-SF-PEJ_21:HRS_DM1AA-SF-PEJ(21)" H 12200 4850 50  0001 L BNN
 F 3 "https://www.hirose.com/product/document?clcode=CL0609-0004-8-72&productname=DM1AA-SF-PEJ(72)&series=DM1&documenttype=Catalog&lang=en&documentid=D31696_en" H 12200 4850 50  0001 L BNN
 F 4 "HRS" H 12200 4850 50  0001 L BNN "MANUFACTURER"
+F 5 "DM1AA-SF-PEJ-21" H 12200 4850 50  0001 C CNN "Component name"
+F 6 "https://www.digikey.no/product-detail/no/hirose-electric-co-ltd/DM1AA-SF-PEJ-21/HR845CT-ND/559985" H 12200 4850 50  0001 C CNN "DK_Detail_Page"
 	1    12200 4850
 	1    0    0    -1
@@
 F 0 "J102" H 12100 2667 50  0000 C CNN
 F 1 "MCU USART1 Header" H 12100 2576 50  0000 C CNN
-F 2 "Connector_PinHeader_2.54mm:PinHeader_2x06_P2.54mm_Vertical" H 12050 2250 50  0001 C CNN
+F 2 "Connector_PinHeader_2.54mm:PinHeader_2x06_P2.54mm_Vertical_SMD" H 12050 2250 50  0001 C CNN
 F 3 "~" H 12050 2250 50  0001 C CNN
+F 4 "0015910120" H 12050 2250 50  0001 C CNN "Component name"
+F 5 "https://www.digikey.no/product-detail/en/molex/0015910120/WM17460-ND/614776" H 12050 2250 50  0001 C CNN "DK_Detail_Page"
 	1    12050 2250
 	1    0    0    -1

Commit message: add final footprint, fix path in footprint library
Parts:
- R105, R106: footprint Resistor_SMD:R_2512_6332Metric_Pad1.40x3.35mm_HandSolder -> tdt4295:RESC6332X120N; Component name (none) -> 352215RFT
Changed lines of the file:
@@
 F 0 "R105" V 9150 3400 50  0000 C CNN
 F 1 "15" V 9100 3200 50  0000 C CNN
-F 2 "Resistor_SMD:R_2512_6332Metric_Pad1.40x3.35mm_HandSolder" V 9030 3200 50  0001 C CNN
+F 2 "tdt4295:RESC6332X120N" V 9030 3200 50  0001 C CNN
 F 3 "https://www.te.com/commerce/DocumentDelivery/DDEController?Action=srchrtrv&DocNm=9-1773463-7&DocType=DS&DocLang=English" H 9100 3200 50  0001 C CNN
 F 4 "352215RFT" H 9100 3200 50  0001 C CNN "Category"
 F 5 "https://www.digikey.no/product-detail/no/te-connectivity-passive-product/352215RFT/A121147CT-ND/5245204" H 9100 3200 50  0001 C CNN "DK_Detail_Page"
+F 6 "352215RFT" H 9100 3200 50  0001 C CNN "Component name"
 	1    9100 3200
 	0    1    1    0
@@
 F 0 "R106" V 9150 3500 50  0000 C CNN
 F 1 "15" V 9100 3300 50  0000 C CNN
-F 2 "Resistor_SMD:R_2512_6332Metric_Pad1.40x3.35mm_HandSolder" V 9030 3300 50  0001 C CNN
+F 2 "tdt4295:RESC6332X120N" V 9030 3300 50  0001 C CNN
 F 3 "https://www.te.com/commerce/DocumentDelivery/DDEController?Action=srchrtrv&DocNm=9-1773463-7&DocType=DS&DocLang=English" H 9100 3300 50  0001 C CNN
 F 4 "352215RFT" H 9100 3300 50  0001 C CNN "Category"
 F 5 "https://www.digikey.no/product-detail/no/te-connectivity-passive-product/352215RFT/A121147CT-ND/5245204" H 9100 3300 50  0001 C CNN "DK_Detail_Page"
+F 6 "352215RFT" H 9100 3300 50  0001 C CNN "Component name"
 	1    9100 3300
 	0    1    1    0

Commit message: minor fixes and import everything into the router
Parts:
- C106, C107: footprint Capacitor_SMD:C_0603_1608Metric_Pad1.08x0.95mm_HandSolder -> Capacitor_SMD:C_0805_2012Metric_Pad1.18x1.45mm_HandSolder
- renumbered R112 to R110, R113 to R111, R114 to R112, R115 to R113
Changed lines of the file:
@@
 F 0 "C107" H 9550 4300 50  0000 L CNN
 F 1 "1uF" H 9550 4100 50  0000 L CNN
-F 2 "Capacitor_SMD:C_0603_1608Metric_Pad1.08x0.95mm_HandSolder" H 9588 4050 50  0001 C CNN
+F 2 "Capacitor_SMD:C_0805_2012Metric_Pad1.18x1.45mm_HandSolder" H 9588 4050 50  0001 C CNN
 F 3 "www.samsungsem.com/kr/support/product-search/mlcc/CL21B105KOFNNNE.jsp" H 9550 4200 50  0001 C CNN
 F 4 "CL21B105KOFNNNE" H 9550 4200 50  0001 C CNN "Component name"
@@
 F 0 "C106" H 9600 3650 50  0000 L CNN
 F 1 "1uF" H 9600 3550 50  0000 L CNN
-F 2 "Capacitor_SMD:C_0603_1608Metric_Pad1.08x0.95mm_HandSolder" H 9538 3450 50  0001 C CNN
+F 2 "Capacitor_SMD:C_0805_2012Metric_Pad1.18x1.45mm_HandSolder" H 9538 3450 50  0001 C CNN
 F 3 "www.samsungsem.com/kr/support/product-search/mlcc/CL21B105KOFNNNE.jsp" H 9500 3600 50  0001 C CNN
 F 4 "CL21B105KOFNNNE" H 9500 3600 50  0001 C CNN "Component name"
@@
 $EndComp
 $Comp
-L Device:R R112
+L Device:R R110
 U 1 1 614E2162
 P 13800 1600
-F 0 "R112" H 13800 1750 50  0000 L CNN
+F 0 "R110" H 13800 1750 50  0000 L CNN
 F 1 "100K" V 13800 1500 50  0000 L CNN
 F 2 "Resistor_SMD:R_0805_2012Metric_Pad1.20x1.40mm_HandSolder" V 13730 1600 50  0001 C CNN
@@
 	15000 2200 15150 2200
 $Comp
-L Device:R R113
+L Device:R R111
 U 1 1 6158865B
 P 14000 1600
-F 0 "R113" H 14000 1750 50  0000 L CNN
+F 0 "R111" H 14000 1750 50  0000 L CNN
 F 1 "100K" V 14000 1500 50  0000 L CNN
 F 2 "Resistor_SMD:R_0805_2012Metric_Pad1.20x1.40mm_HandSolder" V 13930 1600 50  0001 C CNN
@@
 $EndComp
 $Comp
-L Device:R R114
+L Device:R R112
 U 1 1 615889F3
 P 14200 1600
-F 0 "R114" H 14200 1750 50  0000 L CNN
+F 0 "R112" H 14200 1750 50  0000 L CNN
 F 1 "100K" V 14200 1500 50  0000 L CNN
 F 2 "Resistor_SMD:R_0805_2012Metric_Pad1.20x1.40mm_HandSolder" V 14130 1600 50  0001 C CNN
@@
 $EndComp
 $Comp
-L Device:R R115
+L Device:R R113
 U 1 1 61599A1D
 P 14400 1600
-F 0 "R115" H 14400 1750 50  0000 L CNN
+F 0 "R113" H 14400 1750 50  0000 L CNN
 F 1 "100K" V 14400 1500 50  0000 L CNN
 F 2 "Resistor_SMD:R_0805_2012Metric_Pad1.20x1.40mm_HandSolder" V 14330 1600 50  0001 C CNN

Commit message: add digikey part numbers, create BOM
Parts:
- C101, C105, C108, C109, C110: Digi-Key_PN (none) -> 1276-1006-1-ND
- C102: Digi-Key_PN (none) -> 1276-1009-1-ND
- C103, C104, C111: Digi-Key_PN (none) -> 1276-1038-1-ND
- C106, C107: Digi-Key_PN (none) -> 1276-1026-1-ND
- D101, D102, D103, D104: Digi-Key_PN (none) -> 732-4989-1-ND
- J101: Digi-Key_PN (none) -> SAM13960CT-ND
- J102: Digi-Key_PN (none) -> WM17460-ND
- J103: Digi-Key_PN (none) -> HR845CT-ND
- J104: Digi-Key_PN (none) -> WM20569-ND
- R101, R102, R103, R104: Digi-Key_PN (none) -> RHC2512FT330RCT-ND
- R105, R106: Digi-Key_PN (none) -> A121147CT-ND
- R107, R108, R109: footprint Resistor_SMD:R_0805_2012Metric_Pad1.20x1.40mm_HandSolder -> Resistor_SMD:R_1206_3216Metric_Pad1.30x1.75mm_HandSolder; Component name (none) -> RNCP1206FTD100R; Digi-Key_PN (none) -> RNCP1206FTD100RCT-ND
- R110, R111, R112, R113: Digi-Key_PN (none) -> RR12P100KDCT-ND
- U102, U103: Digi-Key_PN (none) -> 1568-1526-ND
