File: pcb/tdt4295/Power_Components.sch (KiCad schematic (older format))
At the start: 43 parts, among them P201 690-005-299-043, U201 TPS54294, U202 TPS54294

Commit message: review stuff
Parts:
- removed D203: IP4220CZ6_125, digikey-footprints:SC-74, symbol dk_TVS-Diodes:IP4220CZ6_125
- added U?: PHDMI2AB4, tdt4295:DFN2510A-10, symbol tdt4295:PHDMI2AB4
- R201, R202: value 1K -> 330
Connections:
- net GND: now also U?.~ (NC)
- net USB_D+: now also U?.~ (NC)
- net USB_D-: now also U?.~ (NC)
- net at C201.1, FB?.2, P201.1: now also U?.~ (NC)
- no-connect marks 8 -> 7
Changed lines of the file:
@@
 	0    -1   1    0
 $EndComp
-Wire Wire Line
-	1250 2150 1900 2150
-$Comp
-L dk_TVS-Diodes:IP4220CZ6_125 D203
-U 1 1 613C398F
-P 2000 3000
-F 0 "D203" V 2053 2520 60  0000 R CNN
-F 1 "IP4220CZ6_125" V 1947 2520 60  0000 R CNN
-F 2 "digikey-footprints:SC-74" H 2200 3200 60  0001 L CNN
-F 3 "https://assets.nexperia.com/documents/data-sheet/IP4220CZ6.pdf" H 2200 3300 60  0001 L CNN
-F 4 "1727-3578-1-ND" H 2200 3400 60  0001 L CNN "Digi-Key_PN"
-F 5 "IP4220CZ6,125" H 2200 3500 60  0001 L CNN "MPN"
-F 6 "Circuit Protection" H 2200 3600 60  0001 L CNN "Category"
-F 7 "TVS - Diodes" H 2200 3700 60  0001 L CNN "Family"
-F 8 "https://assets.nexperia.com/documents/data-sheet/IP4220CZ6.pdf" H 2200 3800 60  0001 L CNN "DK_Datasheet_Link"
-F 9 "/product-detail/en/nexperia-usa-inc/IP4220CZ6,125/1727-3578-1-ND/1133548" H 2200 3900 60  0001 L CNN "DK_Detail_Page"
-F 10 "TVS DIODE 5.5V 6TSOP" H 2200 4000 60  0001 L CNN "Description"
-F 11 "Nexperia USA Inc." H 2200 4100 60  0001 L CNN "Manufacturer"
-F 12 "Active" H 2200 4200 60  0001 L CNN "Status"
-	1    2000 3000
-	0    -1   -1   0
-$EndComp
-Wire Wire Line
-	1050 1750 2100 1750
-Wire Wire Line
-	2100 2500 2100 1750
-Connection ~ 2100 1750
-Wire Wire Line
-	1900 2500 1900 2150
-Connection ~ 1900 2150
-Wire Wire Line
-	1900 2150 2800 2150
-Wire Wire Line
-	2300 2500 2300 2350
 Connection ~ 2300 2350
 Wire Wire Line
@@
 L power:GND #PWR0133
 U 1 1 613C399F
-P 2100 3650
-F 0 "#PWR0133" H 2100 3400 50  0001 C CNN
-F 1 "GND" H 2105 3477 50  0000 C CNN
-F 2 "" H 2100 3650 50  0001 C CNN
-F 3 "" H 2100 3650 50  0001 C CNN
-	1    2100 3650
-	1    0    0    -1
-$EndComp
-Wire Wire Line
-	2100 3500 2100 3650
-NoConn ~ 2300 3600
-NoConn ~ 1900 3600
-Wire Wire Line
-	2300 3500 2300 3600
-Wire Wire Line
-	1900 3600 1900 3500
+P 2100 3600
+F 0 "#PWR0133" H 2100 3350 50  0001 C CNN
+F 1 "GND" H 2105 3427 50  0000 C CNN
+F 2 "" H 2100 3600 50  0001 C CNN
+F 3 "" H 2100 3600 50  0001 C CNN
+	1    2100 3600
+	1    0    0    -1
+$EndComp
 Wire Notes Line
 	3750 4450 650  4450
@@
 P 1000 5750
 F 0 "R201" H 1070 5796 50  0000 L CNN
-F 1 "1K" H 1070 5705 50  0000 L CNN
+F 1 "330" H 1070 5705 50  0000 L CNN
 F 2 "" V 930 5750 50  0001 C CNN
 F 3 "~" H 1000 5750 50  0001 C CNN
@@
 P 1500 5750
 F 0 "R202" H 1570 5796 50  0000 L CNN
-F 1 "1K" H 1570 5705 50  0000 L CNN
+F 1 "330" H 1570 5705 50  0000 L CNN
 F 2 "" V 1430 5750 50  0001 C CNN
 F 3 "~" H 1500 5750 50  0001 C CNN
@@
 	0    1    1    0
 $EndComp
-Wire Wire Line
-	2100 1750 2550 1750
+$Comp
+L tdt4295:PHDMI2AB4 U?
+U 1 1 61657D49
+P 2150 3050
+F 0 "U?" H 1912 2979 50  0000 R CNN
+F 1 "PHDMI2AB4" H 1912 3070 50  0000 R CNN
+F 2 "tdt4295:DFN2510A-10" H 2150 2950 50  0001 C CNN
+F 3 "https://www.google.com/url?sa=t&rct=j&q=&esrc=s&source=web&cd=&ved=2ahUKEwjq-uC3upjzAhUSmYsKHV0iBjEQFnoECAQQAQ&url=https%3A%2F%2Fassets.nexperia.com%2Fdocuments%2Fdata-sheet%2FPHDMI2AB4.pdf&usg=AOvVaw2t6nU9jF_TXAIowSn_9t4X" H 2150 2950 50  0001 C CNN
+	1    2150 3050
+	-1   0    0    1
+$EndComp
+Wire Wire Line
+	2100 3400 2100 3500
+Wire Wire Line
+	2100 3500 1750 3500
+Wire Wire Line
+	1750 3500 1750 2550
+Wire Wire Line
+	1750 2550 2100 2550
+Wire Wire Line
+	2100 2550 2100 2650
+Connection ~ 2100 3500
+Wire Wire Line
+	2100 3500 2100 3600
+Wire Wire Line
+	2300 2350 2300 2650
+Wire Wire Line
+	1050 1750 2200 1750
+Wire Wire Line
+	2200 1750 2200 2650
+Connection ~ 2200 1750
+Wire Wire Line
+	2200 1750 2550 1750
+Wire Wire Line
+	1250 2150 2000 2150
+Wire Wire Line
+	2000 2150 2000 2650
+Connection ~ 2000 2150
+Wire Wire Line
+	2000 2150 2800 2150
+NoConn ~ 1900 2650
 $EndSCHEMATC

Commit message: associate (some) footprints to the symbols
Parts:
- R201, R202: footprint (none) -> Resistor_SMD:R_2512_6332Metric_Pad1.40x3.35mm_HandSolder; Component name (none) -> RHC2512FT330R; DK_Detail_Page (none) -> https://www.digikey.no/product-detail/no/stackpole-electron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
- R203: footprint (none) -> Resistor_SMD:R_0805_2012Metric_Pad1.20x1.40mm_HandSolder; Component name (none) -> RG2012P-3012-B-T5; DK_Detail_Page (none) -> https://www.digikey.no/product-detail/no/susumu/RG2012P-301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
- R204, R207, R209: footprint (none) -> Resistor_SMD:R_0805_2012Metric_Pad1.20x1.40mm_HandSolder; Component name (none) -> RR1220P-2212-D-M; DK_Detail_Page (none) -> https://www.digikey.no/product-detail/no/susumu/RR1220P-221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
- R205: footprint (none) -> Resistor_SMD:R_0805_2012Metric_Pad1.20x1.40mm_HandSolder; Component name (none) -> RR1220P-104-D; DK_Detail_Page (none) -> https://www.digikey.no/product-detail/no/susumu/RR1220P-104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
- R206: footprint (none) -> Resistor_SMD:R_0603_1608Metric_Pad0.98x0.95mm_HandSolder; Component name (none) -> RG1608P-6811-B-T5; DK_Detail_Page (none) -> https://www.digikey.no/product-detail/no/susumu/RG1608P-681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
- R208: footprint (none) -> Resistor_SMD:R_0805_2012Metric_Pad1.20x1.40mm_HandSolder; Component name (none) -> ERA-6AEB7322V; DK_Detail_Page (none) -> https://www.digikey.no/product-detail/no/panasonic-electron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
- U202: renamed from U201; footprint (none) -> tdt4295:TPS54294PWP
- U203: renamed from U202; footprint (none) -> tdt4295:TPS54294PWP
- gave numbers to parts that had none: 2
- renumbered L202 to L201, L203 to L202, L204 to L203

Commit message: pcb: Added some more footprints/part numbers
Parts:
- C205, C206, C214: footprint (none) -> Capacitor_SMD:C_0603_1608Metric_Pad1.08x0.95mm_HandSolder; Component name (none) -> CL10A106KQ8NNNC; DK_Datasheet_Link (none) -> https://www.digikey.no/product-detail/en/samsung-electro-me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
- C210: footprint (none) -> Capacitor_SMD:C_0603_1608Metric_Pad1.08x0.95mm_HandSolder; Component name (none) -> CL21B105KOFNNNE; DK_Datasheet_Link (none) -> https://www.digikey.no/product-detail/en/samsung-electro-me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
- C211: value 1u -> 1uF
- C213: footprint (none) -> Capacitor_SMD:C_0603_1608Metric_Pad1.08x0.95mm_HandSolder; Component name (none) -> CL10B104KA8NNNC; DK_Datasheet_Link (none) -> https://www.digikey.no/product-detail/en/samsung-electro-me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
Changed lines of the file:
@@
 F 0 "C205" H 5115 1796 50  0000 L CNN
 F 1 "10uF" H 5115 1705 50  0000 L CNN
-F 2 "" H 5038 1600 50  0001 C CNN
+F 2 "Capacitor_SMD:C_0603_1608Metric_Pad1.08x0.95mm_HandSolder" H 5038 1600 50  0001 C CNN
 F 3 "~" H 5000 1750 50  0001 C CNN
+F 4 "CL10A106KQ8NNNC" H 5000 1750 50  0001 C CNN "Component name"
+F 5 "https://www.digikey.no/product-detail/en/samsung-electro-mechanics/CL10A106KQ8NNNC/1276-1038-1-ND/3889124" H 5000 1750 50  0001 C CNN "DK_Datasheet_Link"
 	1    5000 1750
 	1    0    0    -1
@@
 F 0 "C206" H 5400 4050 50  0000 L CNN
 F 1 "10uF" H 5400 3850 50  0000 L CNN
-F 2 "" H 5388 3800 50  0001 C CNN
+F 2 "Capacitor_SMD:C_0603_1608Metric_Pad1.08x0.95mm_HandSolder" H 5388 3800 50  0001 C CNN
 F 3 "~" H 5350 3950 50  0001 C CNN
+F 4 "CL10A106KQ8NNNC" H 5350 3950 50  0001 C CNN "Component name"
+F 5 "https://www.digikey.no/product-detail/en/samsung-electro-mechanics/CL10A106KQ8NNNC/1276-1038-1-ND/3889124" H 5350 3950 50  0001 C CNN "DK_Datasheet_Link"
 	1    5350 3950
 	1    0    0    -1
@@
 F 0 "C214" H 9115 3996 50  0000 L CNN
 F 1 "10uF" H 9115 3905 50  0000 L CNN
-F 2 "" H 9038 3800 50  0001 C CNN
+F 2 "Capacitor_SMD:C_0603_1608Metric_Pad1.08x0.95mm_HandSolder" H 9038 3800 50  0001 C CNN
 F 3 "~" H 9000 3950 50  0001 C CNN
+F 4 "CL10A106KQ8NNNC" H 9000 3950 50  0001 C CNN "Component name"
+F 5 "https://www.digikey.no/product-detail/en/samsung-electro-mechanics/CL10A106KQ8NNNC/1276-1038-1-ND/3889124" H 9000 3950 50  0001 C CNN "DK_Datasheet_Link"
 	1    9000 3950
 	1    0    0    -1
@@
 P 8450 4700
 F 0 "C211" H 8500 4800 50  0000 L CNN
-F 1 "1u" H 8500 4600 50  0000 L CNN
+F 1 "1uF" H 8500 4600 50  0000 L CNN
 F 2 "" H 8488 4550 50  0001 C CNN
 F 3 "~" H 8450 4700 50  0001 C CNN
@@
 F 0 "C213" H 8585 1554 50  0000 R CNN
 F 1 "0.1uF" H 8585 1645 50  0000 R CNN
-F 2 "" H 8738 1450 50  0001 C CNN
+F 2 "Capacitor_SMD:C_0603_1608Metric_Pad1.08x0.95mm_HandSolder" H 8738 1450 50  0001 C CNN
 F 3 "~" H 8700 1600 50  0001 C CNN
+F 4 "CL10B104KA8NNNC" H 8700 1600 50  0001 C CNN "Component name"
+F 5 "https://www.digikey.no/product-detail/en/samsung-electro-mechanics/CL10B104KA8NNNC/1276-1006-1-ND/3889092" H 8700 1600 50  0001 C CNN "DK_Datasheet_Link"
 	1    8700 1600
 	-1   0    0    1
@@
 F 0 "C210" H 8315 2596 50  0000 L CNN
 F 1 "1uF" H 8315 2505 50  0000 L CNN
-F 2 "" H 8238 2400 50  0001 C CNN
-F 3 "~" H 8200 2550 50  0001 C CNN
+F 2 "Capacitor_SMD:C_0603_1608Metric_Pad1.08x0.95mm_HandSolder" H 8238 2400 50  0001 C CNN
+F 3 "www.samsungsem.com/kr/support/product-search/mlcc/CL21B105KOFNNNE.jsp" H 8200 2550 50  0001 C CNN
+F 4 "CL21B105KOFNNNE" H 8200 2550 50  0001 C CNN "Component name"
+F 5 "https://www.digikey.no/product-detail/en/samsung-electro-mechanics/CL21B105KOFNNNE/1276-1026-1-ND/3889112" H 8200 2550 50  0001 C CNN "DK_Datasheet_Link"
 	1    8200 2550
 	1    0    0    -1

Commit message: pcb: footprints/components for everything but inductors
Parts:
- C201, C202: footprint (none) -> Capacitor_SMD:C_1210_3225Metric_Pad1.33x2.70mm_HandSolder; Component name (none) -> CL32A107MPVNNNE; DK_Detail_Page (none) -> https://www.digikey.no/product-detail/en/samsung-electro-me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
- C203, C204, C216, C217, C218, C219: footprint (none) -> Capacitor_SMD:C_0603_1608Metric_Pad1.08x0.95mm_HandSolder; Component name (none) -> CL10A226MQ8NRNC; DK_Detail_Page (none) -> https://www.digikey.no/product-detail/en/samsung-electro-me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
- C205, C206, C210, C213, C214: DK_Detail_Page (none) -> https://www.digikey.no/product-detail/en/samsung-electro-me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
- C207, C208, C209, C212, C215: footprint (none) -> Capacitor_SMD:C_0603_1608Metric_Pad1.08x0.95mm_HandSolder; Component name (none) -> CL10B104KA8NNNC; DK_Detail_Page (none) -> https://www.digikey.no/product-detail/en/samsung-electro-me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
- C211: footprint (none) -> Capacitor_SMD:C_0603_1608Metric_Pad1.08x0.95mm_HandSolder; Component name (none) -> CL21B105KOFNNNE; DK_Datasheet_Link (none) -> https://www.digikey.no/product-detail/en/samsung-electro-me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; DK_Detail_Page (none) -> https://www.digikey.no/product-detail/en/samsung-electro-me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
- D201, D202: footprint (none) -> Diode_SMD:D_0805_2012Metric_Pad1.15x1.40mm_HandSolder
- FB201: footprint (none) -> Resistor_SMD:R_0201_0603Metric_Pad0.64x0.40mm_HandSolder; Component name (none) -> BK0603HS330-T; DK_Detail_Page (none) -> https://www.digikey.no/en/products/detail/taiyo-yuden/BK060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; Description (none) -> See fig 2.5 https://www.ftdichip.com/Documents/AppNotes/AN_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

Commit message: pcb: correct vga circuit, modify resistor/capacitor sizes
Parts:
- C207, C208, C209, C212, C215: value 100nF -> 0.1uF
Changed lines of the file:
@@
 P 5450 1750
 F 0 "C207" H 5565 1796 50  0000 L CNN
-F 1 "100nF" H 5565 1705 50  0000 L CNN
+F 1 "0.1uF" H 5565 1705 50  0000 L CNN
 F 2 "Capacitor_SMD:C_0603_1608Metric_Pad1.08x0.95mm_HandSolder" H 5488 1600 50  0001 C CNN
 F 3 "www.samsungsem.com/kr/support/product-search/mlcc/CL21B105KOFNNNE.jsp" H 5450 1750 50  0001 C CNN
@@
 P 5650 3950
 F 0 "C208" H 5750 4050 50  0000 L CNN
-F 1 "100nF" H 5700 3850 50  0000 L CNN
+F 1 "0.1uF" H 5700 3850 50  0000 L CNN
 F 2 "Capacitor_SMD:C_0603_1608Metric_Pad1.08x0.95mm_HandSolder" H 5688 3800 50  0001 C CNN
 F 3 "www.samsungsem.com/kr/support/product-search/mlcc/CL21B105KOFNNNE.jsp" H 5650 3950 50  0001 C CNN
@@
 P 9500 3950
 F 0 "C215" H 9615 3996 50  0000 L CNN
-F 1 "100nF" H 9615 3905 50  0000 L CNN
+F 1 "0.1uF" H 9615 3905 50  0000 L CNN
 F 2 "Capacitor_SMD:C_0603_1608Metric_Pad1.08x0.95mm_HandSolder" H 9538 3800 50  0001 C CNN
 F 3 "www.samsungsem.com/kr/support/product-search/mlcc/CL21B105KOFNNNE.jsp" H 9500 3950 50  0001 C CNN
@@
 P 8650 4150
 F 0 "C212" H 8765 4196 50  0000 L CNN
-F 1 "100nF" H 8765 4105 50  0000 L CNN
+F 1 "0.1uF" H 8765 4105 50  0000 L CNN
 F 2 "Capacitor_SMD:C_0603_1608Metric_Pad1.08x0.95mm_HandSolder" H 8688 4000 50  0001 C CNN
 F 3 "www.samsungsem.com/kr/support/product-search/mlcc/CL21B105KOFNNNE.jsp" H 8650 4150 50  0001 C CNN
@@
 P 6050 4150
 F 0 "C209" H 6100 4250 50  0000 L CNN
-F 1 "100nF" H 6100 4050 50  0000 L CNN
+F 1 "0.1uF" H 6100 4050 50  0000 L CNN
 F 2 "Capacitor_SMD:C_0603_1608Metric_Pad1.08x0.95mm_HandSolder" H 6088 4000 50  0001 C CNN
 F 3 "www.samsungsem.com/kr/support/product-search/mlcc/CL21B105KOFNNNE.jsp" H 6050 4150 50  0001 C CNN

Commit message: add footprints, rename components
Parts:
- C207, C208, C209, C212, C215: DK_Datasheet_Link (none) -> https://www.digikey.no/product-detail/en/samsung-electro-me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
- L201, L203: footprint (none) -> Inductor_SMD:L_1008_2520Metric_Pad1.43x2.20mm_HandSolder; Component name (none) -> TFM252012ALMA1R5MTAA; DK_Detail_Page (none) -> https://www.digikey.no/product-detail/en/tdk-corporation/TF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
- L202: footprint (none) -> Inductor_SMD:L_1008_2520Metric_Pad1.43x2.20mm_HandSolder; Component name (none) -> LQM2HPN2R2MG0L; DK_Detail_Page (none) -> https://www.digikey.no/product-detail/en/murata-electronics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
Changed lines of the file:
@@
 F 4 "CL10B104KA8NNNC" H 5450 1750 50  0001 C CNN "Component name"
 F 5 "https://www.digikey.no/product-detail/en/samsung-electro-mechanics/CL10B104KA8NNNC/1276-1006-1-ND/3889092" H 5450 1750 50  0001 C CNN "DK_Detail_Page"
+F 6 "https://www.digikey.no/product-detail/en/samsung-electro-mechanics/CL10B104KA8NNNC/1276-1006-1-ND/3889092" H 5450 1750 50  0001 C CNN "DK_Datasheet_Link"
 	1    5450 1750
 	1    0    0    -1
@@
 F 0 "L203" V 9640 1400 50  0000 C CNN
 F 1 "1.5uH" V 9549 1400 50  0000 C CNN
-F 2 "" H 9450 1400 50  0001 C CNN
+F 2 "Inductor_SMD:L_1008_2520Metric_Pad1.43x2.20mm_HandSolder" H 9450 1400 50  0001 C CNN
 F 3 "~" H 9450 1400 50  0001 C CNN
+F 4 "TFM252012ALMA1R5MTAA" H 9450 1400 50  0001 C CNN "Component name"
+F 5 "https://www.digikey.no/product-detail/en/tdk-corporation/TFM252012ALMA1R5MTAA/445-175184-6-ND/7795261" H 9450 1400 50  0001 C CNN "DK_Detail_Page"
 	1    9450 1400
 	0    -1   -1   0
@@
 F 4 "CL10B104KA8NNNC" H 5650 3950 50  0001 C CNN "Component name"
 F 5 "https://www.digikey.no/product-detail/en/samsung-electro-mechanics/CL10B104KA8NNNC/1276-1006-1-ND/3889092" H 5650 3950 50  0001 C CNN "DK_Detail_Page"
+F 6 "https://www.digikey.no/product-detail/en/samsung-electro-mechanics/CL10B104KA8NNNC/1276-1006-1-ND/3889092" H 5650 3950 50  0001 C CNN "DK_Datasheet_Link"
 	1    5650 3950
 	1    0    0    -1
@@
 F 4 "CL10B104KA8NNNC" H 9500 3950 50  0001 C CNN "Component name"
 F 5 "https://www.digikey.no/product-detail/en/samsung-electro-mechanics/CL10B104KA8NNNC/1276-1006-1-ND/3889092" H 9500 3950 50  0001 C CNN "DK_Detail_Page"
+F 6 "https://www.digikey.no/product-detail/en/samsung-electro-mechanics/CL10B104KA8NNNC/1276-1006-1-ND/3889092" H 9500 3950 50  0001 C CNN "DK_Datasheet_Link"
 	1    9500 3950
 	1    0    0    -1
@@
 F 4 "CL10B104KA8NNNC" H 8650 4150 50  0001 C CNN "Component name"
 F 5 "https://www.digikey.no/product-detail/en/samsung-electro-mechanics/CL10B104KA8NNNC/1276-1006-1-ND/3889092" H 8650 4150 50  0001 C CNN "DK_Detail_Page"
+F 6 "https://www.digikey.no/product-detail/en/samsung-electro-mechanics/CL10B104KA8NNNC/1276-1006-1-ND/3889092" H 8650 4150 50  0001 C CNN "DK_Datasheet_Link"
 	1    8650 4150
 	1    0    0    -1
@@
 F 0 "L202" V 9440 4300 50  0000 C CNN
 F 1 "2.2uH" V 9349 4300 50  0000 C CNN
-F 2 "" H 9250 4300 50  0001 C CNN
+F 2 "Inductor_SMD:L_1008_2520Metric_Pad1.43x2.20mm_HandSolder" H 9250 4300 50  0001 C CNN
 F 3 "~" H 9250 4300 50  0001 C CNN
+F 4 "LQM2HPN2R2MG0L" H 9250 4300 50  0001 C CNN "Component name"
+F 5 "https://www.digikey.no/product-detail/en/murata-electronics/LQM2HPN2R2MG0L/490-5114-1-ND/1893677" H 9250 4300 50  0001 C CNN "DK_Detail_Page"
 	1    9250 4300
 	0    -1   -1   0
@@
 F 4 "CL10B104KA8NNNC" H 6050 4150 50  0001 C CNN "Component name"
 F 5 "https://www.digikey.no/product-detail/en/samsung-electro-mechanics/CL10B104KA8NNNC/1276-1006-1-ND/3889092" H 6050 4150 50  0001 C CNN "DK_Detail_Page"
+F 6 "https://www.digikey.no/product-detail/en/samsung-electro-mechanics/CL10B104KA8NNNC/1276-1006-1-ND/3889092" H 6050 4150 50  0001 C CNN "DK_Datasheet_Link"
 	1    6050 4150
 	1    0    0    -1
@@
 F 0 "L201" V 5290 4300 50  0000 C CNN
 F 1 "1.5uH" V 5199 4300 50  0000 C CNN
-F 2 "" H 5100 4300 50  0001 C CNN
+F 2 "Inductor_SMD:L_1008_2520Metric_Pad1.43x2.20mm_HandSolder" H 5100 4300 50  0001 C CNN
 F 3 "~" H 5100 4300 50  0001 C CNN
+F 4 "TFM252012ALMA1R5MTAA" H 5100 4300 50  0001 C CNN "Component name"
+F 5 "https://www.digikey.no/product-detail/en/tdk-corporation/TFM252012ALMA1R5MTAA/445-175184-6-ND/7795261" H 5100 4300 50  0001 C CNN "DK_Detail_Page"
 	1    5100 4300
 	0    -1   -1   0
