File: pcb/tdt4295/Power_Components.sch (KiCad schematic (older format))
At the start: 43 parts, among them P201 690-005-299-043, U201 PHDMI2AB4, U202 TPS54294, U203 TPS54294

Commit message: footprints for everything
Parts:
- D201, D202: footprint Diode_SMD:D_0805_2012Metric_Pad1.15x1.40mm_HandSolder -> LED_SMD:LED_0805_2012Metric_Pad1.15x1.40mm_HandSolder
- TP201, TP202, TP203, TP204, TP205: footprint (none) -> TestPoint:TestPoint_Pad_D4.0mm
Changed lines of the file:
@@
 F 0 "D201" V 1039 5232 50  0000 R CNN
 F 1 "LED" V 948 5232 50  0000 R CNN
-F 2 "Diode_SMD:D_0805_2012Metric_Pad1.15x1.40mm_HandSolder" H 1000 5350 50  0001 C CNN
+F 2 "LED_SMD:LED_0805_2012Metric_Pad1.15x1.40mm_HandSolder" H 1000 5350 50  0001 C CNN
 F 3 "~" H 1000 5350 50  0001 C CNN
 	1    1000 5350
@@
 F 0 "D202" V 1539 5232 50  0000 R CNN
 F 1 "LED" V 1448 5232 50  0000 R CNN
-F 2 "Diode_SMD:D_0805_2012Metric_Pad1.15x1.40mm_HandSolder" H 1500 5350 50  0001 C CNN
+F 2 "LED_SMD:LED_0805_2012Metric_Pad1.15x1.40mm_HandSolder" H 1500 5350 50  0001 C CNN
 F 3 "~" H 1500 5350 50  0001 C CNN
 	1    1500 5350
@@
 F 0 "TP201" H 4103 6551 50  0000 L CNN
 F 1 "TestPoint_Probe" H 4103 6460 50  0000 L CNN
-F 2 "" H 4150 6450 50  0001 C CNN
+F 2 "TestPoint:TestPoint_Pad_D4.0mm" H 4150 6450 50  0001 C CNN
 F 3 "~" H 4150 6450 50  0001 C CNN
 	1    3950 6450
@@
 F 0 "TP202" H 4103 6751 50  0000 L CNN
 F 1 "TestPoint_Probe" H 4103 6660 50  0000 L CNN
-F 2 "" H 4150 6650 50  0001 C CNN
+F 2 "TestPoint:TestPoint_Pad_D4.0mm" H 4150 6650 50  0001 C CNN
 F 3 "~" H 4150 6650 50  0001 C CNN
 	1    3950 6650
@@
 F 0 "TP203" H 4103 6951 50  0000 L CNN
 F 1 "TestPoint_Probe" H 4103 6860 50  0000 L CNN
-F 2 "" H 4150 6850 50  0001 C CNN
+F 2 "TestPoint:TestPoint_Pad_D4.0mm" H 4150 6850 50  0001 C CNN
 F 3 "~" H 4150 6850 50  0001 C CNN
 	1    3950 6850
@@
 F 0 "TP204" H 4103 7151 50  0000 L CNN
 F 1 "TestPoint_Probe" H 4103 7060 50  0000 L CNN
-F 2 "" H 4150 7050 50  0001 C CNN
+F 2 "TestPoint:TestPoint_Pad_D4.0mm" H 4150 7050 50  0001 C CNN
 F 3 "~" H 4150 7050 50  0001 C CNN
 	1    3950 7050
@@
 F 0 "TP205" H 4103 7351 50  0000 L CNN
 F 1 "TestPoint_Probe" H 4103 7260 50  0000 L CNN
-F 2 "" H 4150 7250 50  0001 C CNN
+F 2 "TestPoint:TestPoint_Pad_D4.0mm" H 4150 7250 50  0001 C CNN
 F 3 "~" H 4150 7250 50  0001 C CNN
 	1    3950 7250

Commit message: associate component links with (almost) every component
Parts:
- D201: footprint LED_SMD:LED_0805_2012Metric_Pad1.15x1.40mm_HandSolder -> LED_SMD:LED_1206_3216Metric_Pad1.42x1.75mm_HandSolder; Component name (none) -> QTLP650D2TR; DK_Detail_Page (none) -> https://www.digikey.no/product-detail/no/everlight-electron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
- D202: footprint LED_SMD:LED_0805_2012Metric_Pad1.15x1.40mm_HandSolder -> LED_SMD:LED_1206_3216Metric_Pad1.42x1.75mm_HandSolder; Component name (none) -> QTLP650C4TR; DK_Detail_Page (none) -> https://www.digikey.no/product-detail/no/everlight-electron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
- P201: Component name (none) -> 690-005-299-043; DK_Detail_Page /product-detail/en/edac-inc/690-005-299-043/151-1206-1-ND/4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 -> https://www.digikey.no/product-detail/en/edac-inc/690-005-2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
- U201: Component name (none) -> PHDMI2AB4Z; DK_Detail_Page (none) -> https://www.digikey.no/product-detail/no/nexperia-usa-inc/P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
Changed lines of the file:
@@
 F 7 "USB, DVI, HDMI Connectors" H 2150 1300 60  0001 L CNN "Family"
 F 8 "http://files.edac.net/690-005-299-043.pdf" H 2150 1400 60  0001 L CNN "DK_Datasheet_Link"
-F 9 "/product-detail/en/edac-inc/690-005-299-043/151-1206-1-ND/4312192" H 2150 1500 60  0001 L CNN "DK_Detail_Page"
+F 9 "https://www.digikey.no/product-detail/en/edac-inc/690-005-299-043/151-1206-1-ND/4312192" H 2150 1500 60  0001 L CNN "DK_Detail_Page"
 F 10 "CONN RCPT USB2.0 MINI B SMD R/A" H 2150 1600 60  0001 L CNN "Description"
 F 11 "EDAC Inc." H 2150 1700 60  0001 L CNN "Manufacturer"
 F 12 "Active" H 2150 1800 60  0001 L CNN "Status"
+F 13 "690-005-299-043" H 1950 600 50  0001 C CNN "Component name"
 	1    1950 600
 	0    -1   1    0
@@
 F 0 "D201" V 1039 5232 50  0000 R CNN
 F 1 "LED" V 948 5232 50  0000 R CNN
-F 2 "LED_SMD:LED_0805_2012Metric_Pad1.15x1.40mm_HandSolder" H 1000 5350 50  0001 C CNN
+F 2 "LED_SMD:LED_1206_3216Metric_Pad1.42x1.75mm_HandSolder" H 1000 5350 50  0001 C CNN
 F 3 "~" H 1000 5350 50  0001 C CNN
+F 4 "QTLP650D2TR" H 1000 5350 50  0001 C CNN "Component name"
+F 5 "https://www.digikey.no/product-detail/no/everlight-electronics-co-ltd/QTLP650D2TR/1080-1417-1-ND/2676151" H 1000 5350 50  0001 C CNN "DK_Detail_Page"
 	1    1000 5350
 	0    -1   -1   0
@@
 F 0 "D202" V 1539 5232 50  0000 R CNN
 F 1 "LED" V 1448 5232 50  0000 R CNN
-F 2 "LED_SMD:LED_0805_2012Metric_Pad1.15x1.40mm_HandSolder" H 1500 5350 50  0001 C CNN
+F 2 "LED_SMD:LED_1206_3216Metric_Pad1.42x1.75mm_HandSolder" H 1500 5350 50  0001 C CNN
 F 3 "~" H 1500 5350 50  0001 C CNN
+F 4 "QTLP650C4TR" H 1500 5350 50  0001 C CNN "Component name"
+F 5 "https://www.digikey.no/product-detail/no/everlight-electronics-co-ltd/QTLP650C4TR/1080-1415-1-ND/2676149" H 1500 5350 50  0001 C CNN "DK_Detail_Page"
 	1    1500 5350
 	0    -1   -1   0
@@
 F 2 "tdt4295:DFN2510A-10" H 2150 2950 50  0001 C CNN
 F 3 "https://www.google.com/url?sa=t&rct=j&q=&esrc=s&source=web&cd=&ved=2ahUKEwjq-uC3upjzAhUSmYsKHV0iBjEQFnoECAQQAQ&url=https%3A%2F%2Fassets.nexperia.com%2Fdocuments%2Fdata-sheet%2FPHDMI2AB4.pdf&usg=AOvVaw2t6nU9jF_TXAIowSn_9t4X" H 2150 2950 50  0001 C CNN
+F 4 "PHDMI2AB4Z" H 2150 3050 50  0001 C CNN "Component name"
+F 5 "https://www.digikey.no/product-detail/no/nexperia-usa-inc/PHDMI2AB4Z/1727-7820-1-ND/9092244" H 2150 3050 50  0001 C CNN "DK_Detail_Page"
 	1    2150 3050
 	-1   0    0    1

Commit message: minor fixes and import everything into the router
Parts:
- C210, C211: footprint Capacitor_SMD:C_0603_1608Metric_Pad1.08x0.95mm_HandSolder -> Capacitor_SMD:C_0805_2012Metric_Pad1.18x1.45mm_HandSolder
Changed lines of the file:
@@
 F 0 "C211" H 8500 4800 50  0000 L CNN
 F 1 "1uF" H 8500 4600 50  0000 L CNN
-F 2 "Capacitor_SMD:C_0603_1608Metric_Pad1.08x0.95mm_HandSolder" H 8488 4550 50  0001 C CNN
+F 2 "Capacitor_SMD:C_0805_2012Metric_Pad1.18x1.45mm_HandSolder" H 8488 4550 50  0001 C CNN
 F 3 "www.samsungsem.com/kr/support/product-search/mlcc/CL21B105KOFNNNE.jsp" H 8450 4700 50  0001 C CNN
 F 4 "CL21B105KOFNNNE" H 8450 4700 50  0001 C CNN "Component name"
@@
 F 0 "C210" H 8315 2596 50  0000 L CNN
 F 1 "1uF" H 8315 2505 50  0000 L CNN
-F 2 "Capacitor_SMD:C_0603_1608Metric_Pad1.08x0.95mm_HandSolder" H 8238 2400 50  0001 C CNN
+F 2 "Capacitor_SMD:C_0805_2012Metric_Pad1.18x1.45mm_HandSolder" H 8238 2400 50  0001 C CNN
 F 3 "www.samsungsem.com/kr/support/product-search/mlcc/CL21B105KOFNNNE.jsp" H 8200 2550 50  0001 C CNN
 F 4 "CL21B105KOFNNNE" H 8200 2550 50  0001 C CNN "Component name"

Commit message: add digikey part numbers, create BOM
Parts:
- C201, C202: Digi-Key_PN (none) -> 1276-3364-1-ND
- C203, C204, C216, C217, C218, C219: Digi-Key_PN (none) -> 1276-1193-1-ND
- C205, C206, C214: Digi-Key_PN (none) -> 1276-1038-1-ND
- C207, C208, C209, C212, C213, C215: Digi-Key_PN (none) -> 1276-1006-1-ND
- C210, C211: Digi-Key_PN (none) -> 1276-1026-1-ND
- D201: Digi-Key_PN (none) -> 1080-1417-1-ND
- D202: Digi-Key_PN (none) -> 1080-1415-1-ND
- FB201: Digi-Key_PN (none) -> 587-1828-1-ND
- L201, L203: Digi-Key_PN (none) -> 445-175184-1-ND
- L202: Digi-Key_PN (none) -> 490-5114-1-ND
- R201, R202: Digi-Key_PN (none) -> RHC2512FT330RCT-ND
- R203: Digi-Key_PN (none) -> RG20P30.1KBCT-ND
- R204, R207, R209: Digi-Key_PN (none) -> RR12P22.1KDCT-ND
- R205: Digi-Key_PN (none) -> RR12P100KDCT-ND
- R206: Digi-Key_PN (none) -> RG16P6.81KBCT-ND
- R208: Digi-Key_PN (none) -> P73.2KDACT-ND
- U201: Digi-Key_PN (none) -> 1727-7820-1-ND
