File: pcb/tdt4295/fpga.sch (KiCad schematic (older format))
At the start: 45 parts, among them J301 FPGA__debug, U301 S25FL127SABMFV101, U302 NUP4114UCW1T2G, U303 XC7A100T-FTG256-tdt4295

Commit message: pcb: Added some more footprints/part numbers
Parts:
- R312: footprint Resistor_SMD:R_0805_2012Metric_Pad1.20x1.40mm_HandSolder -> Resistor_SMD:R_2512_6332Metric_Pad1.40x3.35mm_HandSolder; Component name RNCF0805TKY200R -> 3521200RFT; DK_Detail_Page https://www.digikey.no/product-detail/no/stackpole-electron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 -> https://www.digikey.no/product-detail/en/te-connectivity-pa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
Changed lines of the file:
@@
 F 0 "R312" H 3270 5646 50  0000 L CNN
 F 1 "200" H 3270 5555 50  0000 L CNN
-F 2 "Resistor_SMD:R_0805_2012Metric_Pad1.20x1.40mm_HandSolder" V 3130 5600 50  0001 C CNN
-F 3 "https://www.seielect.com/catalog/sei-rncf.pdf" H 3200 5600 50  0001 C CNN
-F 4 "RNCF0805TKY200R" H 3200 5600 50  0001 C CNN "Component name"
-F 5 "https://www.digikey.no/product-detail/no/stackpole-electronics-inc/RNCF0805TKY200R/RNCF0805TKY200RCT-ND/4928400" H 3200 5600 50  0001 C CNN "DK_Detail_Page"
+F 2 "Resistor_SMD:R_2512_6332Metric_Pad1.40x3.35mm_HandSolder" V 3130 5600 50  0001 C CNN
+F 3 "https://www.te.com/commerce/DocumentDelivery/DDEController?Action=srchrtrv&DocNm=9-1773463-5&DocType=DS&DocLang=English" H 3200 5600 50  0001 C CNN
+F 4 "3521200RFT" H 3200 5600 50  0001 C CNN "Component name"
+F 5 "https://www.digikey.no/product-detail/en/te-connectivity-passive-product/3521200RFT/A116015CT-ND/4280056" H 3200 5600 50  0001 C CNN "DK_Detail_Page"
 	1    3200 5600
 	1    0    0    -1

Commit message: pcb: footprints/components for everything but inductors
Parts:
- C309: Component name (none) -> CL10A106KQ8NNNC; DK_Detail_Page (none) -> https://www.digikey.no/product-detail/en/samsung-electro-me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
Changed lines of the file:
@@
 F 2 "Capacitor_SMD:C_0805_2012Metric_Pad1.18x1.45mm_HandSolder" H 8138 6100 50  0001 C CNN
 F 3 "~" H 8100 6250 50  0001 C CNN
+F 4 "CL10A106KQ8NNNC" H 8100 6250 50  0001 C CNN "Component name"
+F 5 "https://www.digikey.no/product-detail/en/samsung-electro-mechanics/CL10A106KQ8NNNC/1276-1038-1-ND/3889124" H 8100 6250 50  0001 C CNN "DK_Detail_Page"
 	1    8100 6250
 	1    0    0    -1

Commit message: pcb: correct vga circuit, modify resistor/capacitor sizes
Parts:
- C301: value 100nF -> 0.1uF; footprint Resistor_SMD:R_0402_1005Metric_Pad0.72x0.64mm_HandSolder -> Capacitor_SMD:C_0603_1608Metric_Pad1.08x0.95mm_HandSolder; Component name CL05B104KA5NNNC -> CL10B104KA8NNNC; DK_Detail_Page (none) -> https://www.digikey.no/product-detail/en/samsung-electro-me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
- R301, R302, R305: footprint Resistor_SMD:R_0402_1005Metric_Pad0.72x0.64mm_HandSolder -> Resistor_SMD:R_0805_2012Metric_Pad1.20x1.40mm_HandSolder; DK_Detail_Page https://www.digikey.no/product-detail/no/susumu/RR0510P-102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 -> https://www.digikey.no/product-detail/en/susumu/RR1220P-102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
Changed lines of the file:
@@
 P 1750 1300
 F 0 "C301" H 1865 1346 50  0000 L CNN
-F 1 "100nF" H 1865 1255 50  0000 L CNN
-F 2 "Resistor_SMD:R_0402_1005Metric_Pad0.72x0.64mm_HandSolder" H 1788 1150 50  0001 C CNN
-F 3 "https://media.digikey.com/pdf/Data%20Sheets/Samsung%20PDFs/CL05B104KA5NNNC_Spec.pdf" H 1750 1300 50  0001 C CNN
-F 4 "CL05B104KA5NNNC" H 1750 1300 50  0001 C CNN "Component name"
+F 1 "0.1uF" H 1865 1255 50  0000 L CNN
+F 2 "Capacitor_SMD:C_0603_1608Metric_Pad1.08x0.95mm_HandSolder" H 1788 1150 50  0001 C CNN
+F 3 "" H 1750 1300 50  0001 C CNN
+F 4 "CL10B104KA8NNNC" H 1750 1300 50  0001 C CNN "Component name"
+F 5 "https://www.digikey.no/product-detail/en/samsung-electro-mechanics/CL10B104KA8NNNC/1276-1006-1-ND/3889092" H 1750 1300 50  0001 C CNN "DK_Detail_Page"
 	1    1750 1300
 	1    0    0    -1
@@
 F 0 "R305" V 1930 6850 50  0000 C CNN
 F 1 "1k" V 1850 6850 50  0000 C CNN
-F 2 "Resistor_SMD:R_0402_1005Metric_Pad0.72x0.64mm_HandSolder" V 1780 6850 50  0001 C CNN
+F 2 "Resistor_SMD:R_0805_2012Metric_Pad1.20x1.40mm_HandSolder" V 1780 6850 50  0001 C CNN
 F 3 "https://www.susumu.co.jp/common/pdf/n_catalog_partition05_en.pdf" H 1850 6850 50  0001 C CNN
 F 4 "RR0510P-102-D" H 1850 6850 50  0001 C CNN "Component name"
-F 5 "https://www.digikey.no/product-detail/no/susumu/RR0510P-102-D/RR05P1-0KDCT-ND/432937" H 1850 6850 50  0001 C CNN "DK_Detail_Page"
+F 5 "https://www.digikey.no/product-detail/en/susumu/RR1220P-102-D/RR12P1-0KDCT-ND/432830" H 1850 6850 50  0001 C CNN "DK_Detail_Page"
 	1    1850 6850
 	1    0    0    -1
@@
 F 0 "R302" V 1380 7400 50  0000 C CNN
 F 1 "1k" V 1300 7400 50  0000 C CNN
-F 2 "Resistor_SMD:R_0402_1005Metric_Pad0.72x0.64mm_HandSolder" V 1230 7400 50  0001 C CNN
+F 2 "Resistor_SMD:R_0805_2012Metric_Pad1.20x1.40mm_HandSolder" V 1230 7400 50  0001 C CNN
 F 3 "https://www.susumu.co.jp/common/pdf/n_catalog_partition05_en.pdf" H 1300 7400 50  0001 C CNN
 F 4 "RR0510P-102-D" H 1300 7400 50  0001 C CNN "Component name"
-F 5 "https://www.digikey.no/product-detail/no/susumu/RR0510P-102-D/RR05P1-0KDCT-ND/432937" H 1300 7400 50  0001 C CNN "DK_Detail_Page"
+F 5 "https://www.digikey.no/product-detail/en/susumu/RR1220P-102-D/RR12P1-0KDCT-ND/432830" H 1300 7400 50  0001 C CNN "DK_Detail_Page"
 	1    1300 7400
 	1    0    0    -1
@@
 F 0 "R301" V 930 7400 50  0000 C CNN
 F 1 "1k" V 850 7400 50  0000 C CNN
-F 2 "Resistor_SMD:R_0402_1005Metric_Pad0.72x0.64mm_HandSolder" V 780 7400 50  0001 C CNN
+F 2 "Resistor_SMD:R_0805_2012Metric_Pad1.20x1.40mm_HandSolder" V 780 7400 50  0001 C CNN
 F 3 "https://www.susumu.co.jp/common/pdf/n_catalog_partition05_en.pdf" H 850 7400 50  0001 C CNN
 F 4 "RR0510P-102-D" H 850 7400 50  0001 C CNN "Component name"
-F 5 "https://www.digikey.no/product-detail/no/susumu/RR0510P-102-D/RR05P1-0KDCT-ND/432937" H 850 7400 50  0001 C CNN "DK_Detail_Page"
+F 5 "https://www.digikey.no/product-detail/en/susumu/RR1220P-102-D/RR12P1-0KDCT-ND/432830" H 850 7400 50  0001 C CNN "DK_Detail_Page"
 	1    850  7400
 	1    0    0    -1

Commit message: correct capacitor values, make junctions for IOB34&35
Parts:
- added C?: 330uF, symbol Device:C
- added U?: XC7A100T-FTG256-tdt4295, symbol xc7a100t-ftg256-modified:XC7A100T-FTG256-tdt4295
- C305: value 14pF -> 100uF; footprint Capacitor_SMD:C_1210_3225Metric_Pad1.33x2.70mm_HandSolder -> (none); Component name C1210C107M9PACTU -> (none); DK_Detail_Page https://no.farnell.com/kemet/c1210c107m9pactu/cap-100-f-6-3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 -> (none)
- C308: value 10nF -> 4.7uF; footprint Capacitor_SMD:C_0805_2012Metric_Pad1.18x1.45mm_HandSolder -> (none)
- C309: value 10uF -> 4.7uF; footprint Capacitor_SMD:C_0805_2012Metric_Pad1.18x1.45mm_HandSolder -> (none); Component name CL10A106KQ8NNNC -> (none); DK_Detail_Page https://www.digikey.no/product-detail/en/samsung-electro-me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 -> (none)
Connections:
- net +1V0: now also U303.L8 (VCCINT), C?.1
- net GND: now also U303.F8 (VCCBATT_0), U303.G7 (GNDADC_0), U303.J9 (GND), C?.2, U?.A6 (VCCO_35), U?.B3 (VCCO_35), U?.D7 (VCCO_35), U?.E4 (VCCO_35), U?.F1 (VCCO_35), U?.J2 (VCCO_35), U?.M3 (VCCO_34), U?.R4 (VCCO_34), U?.T1 (VCCO_34)
- net FPGA_DONE: now reaches R312.2, R313.1, U303.H10 (DONE_0)
- net FPGA_PROGRAM_B: now reaches R309.2, U303.L9 (PROGRAM_B_0)
Changed lines of the file:
@@
 P 7800 6250
 F 0 "C308" H 7825 6350 50  0000 L CNN
-F 1 "10nF" H 7825 6150 50  0000 L CNN
-F 2 "Capacitor_SMD:C_0805_2012Metric_Pad1.18x1.45mm_HandSolder" H 7838 6100 50  0001 C CNN
-F 3 "~" H 7800 6250 50  0001 C CNN
+F 1 "4.7uF" H 7825 6150 50  0000 L CNN
+F 2 "" H 7838 6100 50  0001 C CNN
+F 3 "" H 7800 6250 50  0001 C CNN
 	1    7800 6250
 	1    0    0    -1
@@
 P 8100 6250
 F 0 "C309" H 8125 6350 50  0000 L CNN
-F 1 "10uF" H 8125 6150 50  0000 L CNN
-F 2 "Capacitor_SMD:C_0805_2012Metric_Pad1.18x1.45mm_HandSolder" H 8138 6100 50  0001 C CNN
-F 3 "~" H 8100 6250 50  0001 C CNN
-F 4 "CL10A106KQ8NNNC" H 8100 6250 50  0001 C CNN "Component name"
-F 5 "https://www.digikey.no/product-detail/en/samsung-electro-mechanics/CL10A106KQ8NNNC/1276-1038-1-ND/3889124" H 8100 6250 50  0001 C CNN "DK_Detail_Page"
+F 1 "4.7uF" H 8125 6150 50  0000 L CNN
+F 2 "" H 8138 6100 50  0001 C CNN
+F 3 "" H 8100 6250 50  0001 C CNN
+F 4 "" H 8100 6250 50  0001 C CNN "Component name"
+F 5 "" H 8100 6250 50  0001 C CNN "DK_Detail_Page"
 	1    8100 6250
 	1    0    0    -1
@@
 P 7450 5450
 F 0 "C305" H 7475 5550 50  0000 L CNN
-F 1 "14pF" H 7475 5350 50  0000 L CNN
-F 2 "Capacitor_SMD:C_1210_3225Metric_Pad1.33x2.70mm_HandSolder" H 7488 5300 50  0001 C CNN
-F 3 "https://api.kemet.com/component-edge/download/specsheet/C1210C107M9PACTU.pdf" H 7450 5450 50  0001 C CNN
-F 4 "https://no.farnell.com/kemet/c1210c107m9pactu/cap-100-f-6-3v-20-x5r-1210/dp/1108328?st=c1210c107m9pactu" H 7450 5450 50  0001 C CNN "DK_Detail_Page"
-F 5 "C1210C107M9PACTU" H 7450 5450 50  0001 C CNN "Component name"
+F 1 "100uF" H 7475 5350 50  0000 L CNN
+F 2 "" H 7488 5300 50  0001 C CNN
+F 3 "" H 7450 5450 50  0001 C CNN
+F 4 "" H 7450 5450 50  0001 C CNN "DK_Detail_Page"
+F 5 "" H 7450 5450 50  0001 C CNN "Component name"
 	1    7450 5450
 	1    0    0    -1
@@
 Wire Wire Line
 	8850 2250 8850 2350
-Wire Wire Line
-	8850 1450 8850 1650
-Wire Wire Line
-	8900 1450 8850 1450
 Wire Wire Line
 	8850 2250 8900 2250
@@
 Wire Wire Line
 	10850 6100 10550 6100
-Wire Wire Line
-	6600 6100 6600 5900
 Connection ~ 6900 6100
 Wire Wire Line
@@
 Wire Wire Line
 	3650 5150 4000 5150
+Wire Wire Line
+	8900 1450 8850 1450
+Wire Wire Line
+	8850 1450 8850 1650
+Wire Wire Line
+	8850 1650 8850 2150
+Connection ~ 8850 1650
+Connection ~ 8850 2150
+Wire Wire Line
+	10900 1550 10900 1450
+Connection ~ 10900 1450
+Wire Wire Line
+	10900 2150 10900 2250
+Connection ~ 10900 2250
+Text GLabel 2400 6050 0    50   Input ~ 0
+FPGA_PROGRAM_B
+Wire Wire Line
+	3200 5850 2400 5850
+Wire Wire Line
+	2500 6050 2400 6050
+Connection ~ 2500 6050
+Text GLabel 2400 5850 0    50   Input ~ 0
+FPGA_DONE
+Wire Wire Line
+	6600 6100 6600 5900
+$Comp
+L Device:C C?
+U 1 1 615AFA54
+P 6600 6250
+F 0 "C?" H 6625 6350 50  0000 L CNN
+F 1 "330uF" H 6625 6150 50  0000 L CNN
+F 2 "" H 6638 6100 50  0001 C CNN
+F 3 "" H 6600 6250 50  0001 C CNN
+F 4 "" H 6600 6250 50  0001 C CNN "Component name"
+F 5 "" H 6600 6250 50  0001 C CNN "DK_Datasheet_Link"
+F 6 "" H 6600 6250 50  0001 C CNN "DK_Detail_Page"
+	1    6600 6250
+	1    0    0    -1
+$EndComp
+Connection ~ 6600 6100
+Connection ~ 6600 6400
+Wire Wire Line
+	9800 3900 9800 4000
+Connection ~ 9800 4000
+Wire Wire Line
+	9800 4000 9800 4100
+Connection ~ 9800 4100
+Wire Wire Line
+	9800 4100 9800 4250
+Connection ~ 9800 4250
+Wire Wire Line
+	9800 4250 9800 4350
+Connection ~ 9800 4350
+Wire Wire Line
+	9800 4350 9800 4450
+Connection ~ 9800 4450
+Wire Wire Line
+	9800 4450 9800 4550
+Connection ~ 9800 4550
+Wire Wire Line
+	9800 4550 9800 4650
+Connection ~ 9800 4650
+Wire Wire Line
+	9800 4650 9800 4750
+$Comp
+L xc7a100t-ftg256-modified:XC7A100T-FTG256-tdt4295 U?
+U 7 1 615C8949
+P 10300 4350
+F 0 "U?" H 10200 3800 50  0000 L CNN
+F 1 "XC7A100T-FTG256-tdt4295" H 9800 3700 50  0000 L CNN
+F 2 "" H 10300 1300 50  0001 C CNN
+F 3 "" H 10300 1300 50  0000 C CNN
+	7    10300 4350
+	1    0    0    -1
+$EndComp
+$Comp
+L power:GND #PWR?
+U 1 1 615F9D9F
+P 9800 4750
+F 0 "#PWR?" H 9800 4500 50  0001 C CNN
+F 1 "GND" H 9805 4577 50  0000 C CNN
+F 2 "" H 9800 4750 50  0001 C CNN
+F 3 "" H 9800 4750 50  0001 C CNN
+	1    9800 4750
+	1    0    0    -1
+$EndComp
+Connection ~ 9800 4750
 $EndSCHEMATC
