File: pcb/tdt4295/fpga_iob14.sch (KiCad schematic (older format))
At the start: 10 parts, among them U303 XC7A100T-FTG256-tdt4295, U601 DSC1001AL5-100.0000

Commit message: add footprints, rename components
Parts:
- C601: DK_Datasheet_Link (none) -> https://www.digikey.no/product-detail/en/samsung-electro-me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
- C605, C606, C607, C608: DK_Detail_Page (none) -> https://www.digikey.no/product-detail/en/murata-electronics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
Changed lines of the file:
@@
 F 3 "https://www.farnell.com/datasheets/2048812.pdf" H 8150 1100 50  0001 C CNN
 F 4 "GRM188R71C474KA88D" H 8150 1100 50  0001 C CNN "Component name"
+F 5 "https://www.digikey.no/product-detail/en/murata-electronics/GRM188R71C474KA88D/490-3295-1-ND/702836" H 8150 1100 50  0001 C CNN "DK_Detail_Page"
 	1    8150 1100
 	1    0    0    -1
@@
 F 3 "https://www.farnell.com/datasheets/2048812.pdf" H 8500 1100 50  0001 C CNN
 F 4 "GRM188R71C474KA88D" H 8500 1100 50  0001 C CNN "Component name"
+F 5 "https://www.digikey.no/product-detail/en/murata-electronics/GRM188R71C474KA88D/490-3295-1-ND/702836" H 8500 1100 50  0001 C CNN "DK_Detail_Page"
 	1    8500 1100
 	1    0    0    -1
@@
 F 3 "https://www.farnell.com/datasheets/2048812.pdf" H 8900 1100 50  0001 C CNN
 F 4 "GRM188R71C474KA88D" H 8900 1100 50  0001 C CNN "Component name"
+F 5 "https://www.digikey.no/product-detail/en/murata-electronics/GRM188R71C474KA88D/490-3295-1-ND/702836" H 8900 1100 50  0001 C CNN "DK_Detail_Page"
 	1    8900 1100
 	1    0    0    -1
@@
 F 3 "https://www.farnell.com/datasheets/2048812.pdf" H 9250 1100 50  0001 C CNN
 F 4 "GRM188R71C474KA88D" H 9250 1100 50  0001 C CNN "Component name"
+F 5 "https://www.digikey.no/product-detail/en/murata-electronics/GRM188R71C474KA88D/490-3295-1-ND/702836" H 9250 1100 50  0001 C CNN "DK_Detail_Page"
 	1    9250 1100
 	1    0    0    -1
@@
 F 4 "CL10B104KA8NNNC" H 850 1350 50  0001 C CNN "Component name"
 F 5 "https://www.digikey.no/product-detail/en/samsung-electro-mechanics/CL10B104KA8NNNC/1276-1006-1-ND/3889092" H 850 1350 50  0001 C CNN "DK_Detail_Page"
+F 6 "https://www.digikey.no/product-detail/en/samsung-electro-mechanics/CL10B104KA8NNNC/1276-1006-1-ND/3889092" H 850 1350 50  0001 C CNN "DK_Datasheet_Link"
 	1    850  1350
 	-1   0    0    1
@@
 	9600 950  9600 800
 $Comp
-L power:GND #PWR0605
+L power:GND #PWR0606
 U 1 1 614B3B58
 P 9600 1350
-F 0 "#PWR0605" H 9600 1100 50  0001 C CNN
+F 0 "#PWR0606" H 9600 1100 50  0001 C CNN
 F 1 "GND" H 9605 1177 50  0000 C CNN
 F 2 "" H 9600 1350 50  0001 C CNN
@@
 $EndComp
 $Comp
-L power:+3V3 #PWR0604
+L power:+3V3 #PWR0605
 U 1 1 614741B9
 P 9600 800
-F 0 "#PWR0604" H 9600 650 50  0001 C CNN
+F 0 "#PWR0605" H 9600 650 50  0001 C CNN
 F 1 "+3V3" H 9450 850 50  0000 C CNN
 F 2 "" H 9600 800 50  0001 C CNN
@@
 	5200 2250 4750 2250
 $Comp
-L power:GND #PWR?
+L power:GND #PWR0604
 U 1 1 6158A76A
 P 4750 2250
-F 0 "#PWR?" H 4750 2000 50  0001 C CNN
+F 0 "#PWR0604" H 4750 2000 50  0001 C CNN
 F 1 "GND" H 4755 2077 50  0000 C CNN
 F 2 "" H 4750 2250 50  0001 C CNN

Commit message: associate component links with (almost) every component
Parts:
- U601: Component name (none) -> DSC1001AL5-100.0000; DK_Detail_Page (none) -> https://www.digikey.no/product-detail/no/microchip-technolo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
Changed lines of the file:
@@
 F 2 "DSC1001AL5-100.0000:DSC1001AL5-100.0000" H 2250 1990 60  0001 C CNN
 F 3 "https://rocelec.widen.net/view/pdf/4jp9qpy8qv/MCHP-S-A0003587227-1.pdf?t.download=true&u=5oefqw" H 1250 1750 60  0001 C CNN
+F 4 "DSC1001AL5-100.0000" H 1250 1750 50  0001 C CNN "Component name"
+F 5 "https://www.digikey.no/product-detail/no/microchip-technology/DSC1001AL5-100-0000/DSC1001AL5-100-0000-ND/5773489" H 1250 1750 50  0001 C CNN "DK_Detail_Page"
 	1    1250 1750
 	1    0    0    -1

Commit message: add digikey part numbers, create BOM
Parts:
- C601: Digi-Key_PN (none) -> 1276-1006-1-ND
- C602: Digi-Key_PN (none) -> 490-6543-1-ND
- C603, C604: Digi-Key_PN (none) -> 445-7591-1-ND
- C605, C606, C607, C608: Digi-Key_PN (none) -> 490-3295-1-ND
- U601: Digi-Key_PN (none) -> DSC1001AL5-100.0000-ND
Changed lines of the file:
@@
 F 4 "GRM32ER71A476ME15L" H 7150 1100 50  0001 C CNN "Component name"
 F 5 "https://www.digikey.no/product-detail/no/murata-electronics/GRM32ER71A476ME15L/490-6543-1-ND/3845740" H 7150 1100 50  0001 C CNN "DK_Detail_Page"
+F 6 "490-6543-1-ND" H 7150 1100 50  0001 C CNN "Digi-Key_PN"
 	1    7150 1100
 	1    0    0    -1
@@
 F 5 "" H 7450 1100 50  0001 C CNN "DK_Datasheet_Link"
 F 6 "https://www.digikey.no/product-detail/no/tdk-corporation/C2012X7R1A475K125AC/445-7591-1-ND/2733663" H 7450 1100 50  0001 C CNN "DK_Detail_Page"
+F 7 "445-7591-1-ND" H 7450 1100 50  0001 C CNN "Digi-Key_PN"
 	1    7450 1100
 	1    0    0    -1
@@
 F 5 "" H 7800 1100 50  0001 C CNN "DK_Datasheet_Link"
 F 6 "https://www.digikey.no/product-detail/no/tdk-corporation/C2012X7R1A475K125AC/445-7591-1-ND/2733663" H 7800 1100 50  0001 C CNN "DK_Detail_Page"
+F 7 "445-7591-1-ND" H 7800 1100 50  0001 C CNN "Digi-Key_PN"
 	1    7800 1100
 	1    0    0    -1
@@
 F 4 "GRM188R71C474KA88D" H 8150 1100 50  0001 C CNN "Component name"
 F 5 "https://www.digikey.no/product-detail/en/murata-electronics/GRM188R71C474KA88D/490-3295-1-ND/702836" H 8150 1100 50  0001 C CNN "DK_Detail_Page"
+F 6 "490-3295-1-ND" H 8150 1100 50  0001 C CNN "Digi-Key_PN"
 	1    8150 1100
 	1    0    0    -1
@@
 F 4 "GRM188R71C474KA88D" H 8500 1100 50  0001 C CNN "Component name"
 F 5 "https://www.digikey.no/product-detail/en/murata-electronics/GRM188R71C474KA88D/490-3295-1-ND/702836" H 8500 1100 50  0001 C CNN "DK_Detail_Page"
+F 6 "490-3295-1-ND" H 8500 1100 50  0001 C CNN "Digi-Key_PN"
 	1    8500 1100
 	1    0    0    -1
@@
 F 4 "GRM188R71C474KA88D" H 8900 1100 50  0001 C CNN "Component name"
 F 5 "https://www.digikey.no/product-detail/en/murata-electronics/GRM188R71C474KA88D/490-3295-1-ND/702836" H 8900 1100 50  0001 C CNN "DK_Detail_Page"
+F 6 "490-3295-1-ND" H 8900 1100 50  0001 C CNN "Digi-Key_PN"
 	1    8900 1100
 	1    0    0    -1
@@
 F 4 "GRM188R71C474KA88D" H 9250 1100 50  0001 C CNN "Component name"
 F 5 "https://www.digikey.no/product-detail/en/murata-electronics/GRM188R71C474KA88D/490-3295-1-ND/702836" H 9250 1100 50  0001 C CNN "DK_Detail_Page"
+F 6 "490-3295-1-ND" H 9250 1100 50  0001 C CNN "Digi-Key_PN"
 	1    9250 1100
 	1    0    0    -1
@@
 F 4 "DSC1001AL5-100.0000" H 1250 1750 50  0001 C CNN "Component name"
 F 5 "https://www.digikey.no/product-detail/no/microchip-technology/DSC1001AL5-100-0000/DSC1001AL5-100-0000-ND/5773489" H 1250 1750 50  0001 C CNN "DK_Detail_Page"
+F 6 "DSC1001AL5-100.0000-ND" H 1250 1750 50  0001 C CNN "Digi-Key_PN"
 	1    1250 1750
 	1    0    0    -1
@@
 F 5 "https://www.digikey.no/product-detail/en/samsung-electro-mechanics/CL10B104KA8NNNC/1276-1006-1-ND/3889092" H 850 1350 50  0001 C CNN "DK_Detail_Page"
 F 6 "https://www.digikey.no/product-detail/en/samsung-electro-mechanics/CL10B104KA8NNNC/1276-1006-1-ND/3889092" H 850 1350 50  0001 C CNN "DK_Datasheet_Link"
+F 7 "1276-1006-1-ND" H 850 1350 50  0001 C CNN "Digi-Key_PN"
 	1    850  1350
 	-1   0    0    1
