File: pcb/tdt4295/fpga_ext_IO.sch (KiCad schematic (older format))
At the start: 44 parts, among them J501 618015330923, J502 FPGA GPIO, U501 NUP4114UCW1T2G, U502 NUP4114UCW1T2G, U503 NUP4114UCW1T2G, U504 NUP4114UCW1T2G

Commit message: correct 330 Ohm footprints, route some more FPGA
Parts:
- R507, R508, R509, R510: footprint Resistor_SMD:R_0805_2012Metric_Pad1.20x1.40mm_HandSolder -> Resistor_SMD:R_2512_6332Metric_Pad1.40x3.35mm_HandSolder; Component name RK73H2ATTD3300F -> RHC2512FT330R
- R518, R519: footprint Resistor_SMD:R_0805_2012Metric_Pad1.20x1.40mm_HandSolder -> Resistor_SMD:R_1206_3216Metric_Pad1.30x1.75mm_HandSolder
- U501, U502, U503, U504: symbol NUP4114UCW1T2G:NUP4114UCW1T2G -> tdt4295-rescue:NUP4114UCW1T2G-NUP4114UCW1T2G
Changed lines of the file:
@@
 $Descr A4 11693 8268
 encoding utf-8
-Sheet 5 6
+Sheet 3 6
 Title ""
 Date ""
@@
 F 0 "R508" V 1430 1250 50  0000 C CNN
 F 1 "330" V 1350 1250 50  0000 C CNN
-F 2 "Resistor_SMD:R_0805_2012Metric_Pad1.20x1.40mm_HandSolder" V 1280 1250 50  0001 C CNN
+F 2 "Resistor_SMD:R_2512_6332Metric_Pad1.40x3.35mm_HandSolder" V 1280 1250 50  0001 C CNN
 F 3 "https://www.koaspeer.com/pdfs/RK73H.pdf" H 1350 1250 50  0001 C CNN
-F 4 "RK73H2ATTD3300F" H 1350 1250 50  0001 C CNN "Component name"
+F 4 "RHC2512FT330R" H 1350 1250 50  0001 C CNN "Component name"
 F 5 "https://www.digikey.no/product-detail/no/koa-speer-electronics-inc/RK73H2ATTD3300F/2019-RK73H2ATTD3300FCT-ND/10235463" H 1350 1250 50  0001 C CNN "DK_Detail_Page"
 	1    1350 1250
@@
 AR Path="/61537853/615B3EE9" Ref="R?"  Part="1"
 AR Path="/617F72AC/61537853/615B3EE9" Ref="R501"  Part="1"
-F 0 "R501" V 1400 4500 50  0000 C CNN
+F 0 "R?" V 1400 4500 50  0000 C CNN
 F 1 "4k" V 1300 4500 50  0000 C CNN
 F 2 "Resistor_SMD:R_1206_3216Metric_Pad1.30x1.75mm_HandSolder" V 1230 4500 50  0001 C CNN
@@
 AR Path="/61537853/615EF461" Ref="R?"  Part="1"
 AR Path="/617F72AC/61537853/615EF461" Ref="R503"  Part="1"
-F 0 "R503" V 1400 5150 50  0000 C CNN
+F 0 "R?" V 1400 5150 50  0000 C CNN
 F 1 "4k" V 1300 5150 50  0000 C CNN
 F 2 "Resistor_SMD:R_1206_3216Metric_Pad1.30x1.75mm_HandSolder" V 1230 5150 50  0001 C CNN
@@
 AR Path="/61537853/615FE017" Ref="R?"  Part="1"
 AR Path="/617F72AC/61537853/615FE017" Ref="R505"  Part="1"
-F 0 "R505" V 1400 5850 50  0000 C CNN
+F 0 "R?" V 1400 5850 50  0000 C CNN
 F 1 "4k" V 1300 5850 50  0000 C CNN
 F 2 "Resistor_SMD:R_1206_3216Metric_Pad1.30x1.75mm_HandSolder" V 1230 5850 50  0001 C CNN
@@
 F 0 "R507" V 1430 900 50  0000 C CNN
 F 1 "330" V 1350 900 50  0000 C CNN
-F 2 "Resistor_SMD:R_0805_2012Metric_Pad1.20x1.40mm_HandSolder" V 1280 900 50  0001 C CNN
+F 2 "Resistor_SMD:R_2512_6332Metric_Pad1.40x3.35mm_HandSolder" V 1280 900 50  0001 C CNN
 F 3 "https://www.koaspeer.com/pdfs/RK73H.pdf" H 1350 900 50  0001 C CNN
-F 4 "RK73H2ATTD3300F" H 1350 900 50  0001 C CNN "Component name"
+F 4 "RHC2512FT330R" H 1350 900 50  0001 C CNN "Component name"
 F 5 "https://www.digikey.no/product-detail/no/koa-speer-electronics-inc/RK73H2ATTD3300F/2019-RK73H2ATTD3300FCT-ND/10235463" H 1350 900 50  0001 C CNN "DK_Detail_Page"
 	1    1350 900
@@
 F 0 "R509" V 1430 1600 50  0000 C CNN
 F 1 "330" V 1350 1600 50  0000 C CNN
-F 2 "Resistor_SMD:R_0805_2012Metric_Pad1.20x1.40mm_HandSolder" V 1280 1600 50  0001 C CNN
+F 2 "Resistor_SMD:R_2512_6332Metric_Pad1.40x3.35mm_HandSolder" V 1280 1600 50  0001 C CNN
 F 3 "https://www.koaspeer.com/pdfs/RK73H.pdf" H 1350 1600 50  0001 C CNN
-F 4 "RK73H2ATTD3300F" H 1350 1600 50  0001 C CNN "Component name"
+F 4 "RHC2512FT330R" H 1350 1600 50  0001 C CNN "Component name"
 F 5 "https://www.digikey.no/product-detail/no/koa-speer-electronics-inc/RK73H2ATTD3300F/2019-RK73H2ATTD3300FCT-ND/10235463" H 1350 1600 50  0001 C CNN "DK_Detail_Page"
 	1    1350 1600
@@
 F 0 "R510" V 1430 1950 50  0000 C CNN
 F 1 "330" V 1350 1950 50  0000 C CNN
-F 2 "Resistor_SMD:R_0805_2012Metric_Pad1.20x1.40mm_HandSolder" V 1280 1950 50  0001 C CNN
+F 2 "Resistor_SMD:R_2512_6332Metric_Pad1.40x3.35mm_HandSolder" V 1280 1950 50  0001 C CNN
 F 3 "https://www.koaspeer.com/pdfs/RK73H.pdf" H 1350 1950 50  0001 C CNN
-F 4 "RK73H2ATTD3300F" H 1350 1950 50  0001 C CNN "Component name"
+F 4 "RHC2512FT330R" H 1350 1950 50  0001 C CNN "Component name"
 F 5 "https://www.digikey.no/product-detail/no/koa-speer-electronics-inc/RK73H2ATTD3300F/2019-RK73H2ATTD3300FCT-ND/10235463" H 1350 1950 50  0001 C CNN "DK_Detail_Page"
 	1    1350 1950
@@
 VGA output
 $Comp
-L NUP4114UCW1T2G:NUP4114UCW1T2G U501
+L tdt4295-rescue:NUP4114UCW1T2G-NUP4114UCW1T2G U501
 U 1 1 61ADFC51
 P 5650 2900
+AR Path="/61ADFC51" Ref="U501"  Part="1"
+AR Path="/617F72AC/61537853/61ADFC51" Ref="U501"  Part="1"
 F 0 "U501" H 5650 2600 60  0000 C CNN
 F 1 "NUP4114UCW1T2G" H 5650 2500 60  0000 C CNN
@@
 $EndComp
 $Comp
-L NUP4114UCW1T2G:NUP4114UCW1T2G U502
+L tdt4295-rescue:NUP4114UCW1T2G-NUP4114UCW1T2G U502
 U 1 1 61B06D56
 P 5800 1100
+AR Path="/61B06D56" Ref="U502"  Part="1"
+AR Path="/617F72AC/61537853/61B06D56" Ref="U502"  Part="1"
 F 0 "U502" H 5800 1650 60  0000 C CNN
 F 1 "NUP4114UCW1T2G" H 5800 1550 60  0000 C CNN
@@
 FPGA_EXT_IO13
 $Comp
-L NUP4114UCW1T2G:NUP4114UCW1T2G U504
+L tdt4295-rescue:NUP4114UCW1T2G-NUP4114UCW1T2G U504
 U 1 1 61B47BBA
 P 8000 3200
+AR Path="/61B47BBA" Ref="U504"  Part="1"
+AR Path="/617F72AC/61537853/61B47BBA" Ref="U504"  Part="1"
 F 0 "U504" H 8000 2900 60  0000 C CNN
 F 1 "NUP4114UCW1T2G" H 8000 2800 60  0000 C CNN
@@
 	7050 2250 7400 2250
 $Comp
-L NUP4114UCW1T2G:NUP4114UCW1T2G U503
+L tdt4295-rescue:NUP4114UCW1T2G-NUP4114UCW1T2G U503
 U 1 1 61BB530D
 P 8000 1100
+AR Path="/61BB530D" Ref="U503"  Part="1"
+AR Path="/617F72AC/61537853/61BB530D" Ref="U503"  Part="1"
 F 0 "U503" H 8000 800 60  0000 C CNN
 F 1 "NUP4114UCW1T2G" H 8000 700 60  0000 C CNN
@@
 F 0 "R519" V 3980 5550 50  0000 C CNN
 F 1 "100" V 3900 5550 50  0000 C CNN
-F 2 "Resistor_SMD:R_0805_2012Metric_Pad1.20x1.40mm_HandSolder" V 3830 5550 50  0001 C CNN
+F 2 "Resistor_SMD:R_1206_3216Metric_Pad1.30x1.75mm_HandSolder" V 3830 5550 50  0001 C CNN
 F 3 "https://www.vishay.com/docs/28758/tnpw_e3.pdf" H 3900 5550 50  0001 C CNN
 F 4 "TNPW0805100RBEEA" H 3900 5550 50  0001 C CNN "Component name"
@@
 F 0 "R518" V 3580 5350 50  0000 C CNN
 F 1 "100" V 3500 5350 50  0000 C CNN
-F 2 "Resistor_SMD:R_0805_2012Metric_Pad1.20x1.40mm_HandSolder" V 3430 5350 50  0001 C CNN
+F 2 "Resistor_SMD:R_1206_3216Metric_Pad1.30x1.75mm_HandSolder" V 3430 5350 50  0001 C CNN
 F 3 "https://www.vishay.com/docs/28758/tnpw_e3.pdf" H 3500 5350 50  0001 C CNN
 F 4 "TNPW0805100RBEEA" H 3500 5350 50  0001 C CNN "Component name"
